File: hardware/pcb/chess-board.kicad_pcb (KiCad board)
At the start: 2 copper layers, 320 x 360 mm, 228 parts, among them J1 2x20 2.54 mm THT, J2 1x4 2.54 mm THT, J3 5.5x2.1 mm THT, SW1 6x6 mm THT, SW10 6x6 mm THT, SW11 6x6 mm THT, SW12 6x6 mm THT, SW13 SPST rocker THT, SW2 6x6 mm THT, SW3 6x6 mm THT, SW4 6x6 mm THT, SW5 6x6 mm THT, SW6 6x6 mm THT, SW7 6x6 mm THT, SW8 6x6 mm THT, SW9 6x6 mm THT, U1 PDIP-28, U10 PLCC-6 5050, U11 PLCC-6 5050, U12 PLCC-6 5050, U13 PLCC-6 5050, U14 PLCC-6 5050, U15 PLCC-6 5050, U16 PLCC-6 5050, U17 PLCC-6 5050, U18 PLCC-6 5050, U19 PLCC-6 5050, U2 PDIP-28, U20 PLCC-6 5050, U21 PLCC-6 5050, U22 PLCC-6 5050, U23 PLCC-6 5050, U24 PLCC-6 5050, U25 PLCC-6 5050, U26 PLCC-6 5050, U27 PLCC-6 5050, U28 PLCC-6 5050, U29 PLCC-6 5050, U3 PDIP-28, U30 PLCC-6 5050, U31 PLCC-6 5050, U32 PLCC-6 5050, U33 PLCC-6 5050, U34 PLCC-6 5050, U35 PLCC-6 5050, U36 PLCC-6 5050, U37 PLCC-6 5050, U38 PLCC-6 5050, U39 PLCC-6 5050, U4 PDIP-28, U40 PLCC-6 5050, U41 PLCC-6 5050, U42 PLCC-6 5050, U43 PLCC-6 5050, U44 PLCC-6 5050, U45 PLCC-6 5050, U46 PLCC-6 5050, U47 PLCC-6 5050, U48 PLCC-6 5050, U49 PLCC-6 5050, U5 DIP-14, U50 PLCC-6 5050, U51 PLCC-6 5050, U52 PLCC-6 5050, U53 PLCC-6 5050, U54 PLCC-6 5050, U55 PLCC-6 5050, U56 PLCC-6 5050, U57 PLCC-6 5050, U58 PLCC-6 5050, U59 PLCC-6 5050, U6 PLCC-6 5050, U60 PLCC-6 5050, U61 PLCC-6 5050, U62 PLCC-6 5050, U63 PLCC-6 5050, U64 PLCC-6 5050, U65 PLCC-6 5050, U66 PLCC-6 5050, U67 PLCC-6 5050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

Commit message: feat(pcb): add four-layer power distribution
Routing:
- net GND: track 0.00 -> 64.0 mm, vias 0 -> 64
- net +5V: track 0.00 -> 64.0 mm, vias 0 -> 64
- added copper zone on In2.Cu, net +5V
- added copper zone on In1.Cu, net GND
Other:
- copper layers 2 -> 4

Commit message: feat(pcb): route regular LED chain links
Routing:
- net LED_D32: track 0.00 -> 55.6 mm, vias 0 -> 2
- net LED_D16: track 0.00 -> 55.6 mm, vias 0 -> 2
- net LED_D48: track 0.00 -> 55.6 mm, vias 0 -> 2
- net LED_C48: track 0.00 -> 54.4 mm
- net LED_C32: track 0.00 -> 54.4 mm
- net LED_C16: track 0.00 -> 54.4 mm
- net LED_C56: track 0.00 -> 47.6 mm
- net LED_C8: track 0.00 -> 47.6 mm
- net LED_C40: track 0.00 -> 47.6 mm
- net LED_C24: track 0.00 -> 47.6 mm
- net LED_D56: track 0.00 -> 42.4 mm, vias 0 -> 2
- net LED_D8: track 0.00 -> 42.4 mm, vias 0 -> 2
- net LED_D40: track 0.00 -> 42.4 mm, vias 0 -> 2
- net LED_D24: track 0.00 -> 42.4 mm, vias 0 -> 2
- net N$241: track 0.00 -> 35.0 mm
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