File: hardware/pcb/chess-board.kicad_pcb (KiCad board)
At the start: 4 copper layers, 320 x 360 mm, 228 parts, among them J1 2x20 2.54 mm THT, J2 1x4 2.54 mm THT, J3 5.5x2.1 mm THT, SW1 6x6 mm THT, SW10 6x6 mm THT, SW11 6x6 mm THT, SW12 6x6 mm THT, SW13 SPST rocker THT, SW2 6x6 mm THT, SW3 6x6 mm THT, SW4 6x6 mm THT, SW5 6x6 mm THT, SW6 6x6 mm THT, SW7 6x6 mm THT, SW8 6x6 mm THT, SW9 6x6 mm THT, U1 PDIP-28, U10 PLCC-6 5050, U11 PLCC-6 5050, U12 PLCC-6 5050, U13 PLCC-6 5050, U14 PLCC-6 5050, U15 PLCC-6 5050, U16 PLCC-6 5050, U17 PLCC-6 5050, U18 PLCC-6 5050, U19 PLCC-6 5050, U2 PDIP-28, U20 PLCC-6 5050, U21 PLCC-6 5050, U22 PLCC-6 5050, U23 PLCC-6 5050, U24 PLCC-6 5050, U25 PLCC-6 5050, U26 PLCC-6 5050, U27 PLCC-6 5050, U28 PLCC-6 5050, U29 PLCC-6 5050, U3 PDIP-28, U30 PLCC-6 5050, U31 PLCC-6 5050, U32 PLCC-6 5050, U33 PLCC-6 5050, U34 PLCC-6 5050, U35 PLCC-6 5050, U36 PLCC-6 5050, U37 PLCC-6 5050, U38 PLCC-6 5050, U39 PLCC-6 5050, U4 PDIP-28, U40 PLCC-6 5050, U41 PLCC-6 5050, U42 PLCC-6 5050, U43 PLCC-6 5050, U44 PLCC-6 5050, U45 PLCC-6 5050, U46 PLCC-6 5050, U47 PLCC-6 5050, U48 PLCC-6 5050, U49 PLCC-6 5050, U5 DIP-14, U50 PLCC-6 5050, U51 PLCC-6 5050, U52 PLCC-6 5050, U53 PLCC-6 5050, U54 PLCC-6 5050, U55 PLCC-6 5050, U56 PLCC-6 5050, U57 PLCC-6 5050, U58 PLCC-6 5050, U59 PLCC-6 5050, U6 PLCC-6 5050, U60 PLCC-6 5050, U61 PLCC-6 5050, U62 PLCC-6 5050, U63 PLCC-6 5050, U64 PLCC-6 5050, U65 PLCC-6 5050, U66 PLCC-6 5050, U67 PLCC-6 5050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

Commit message: feat(hardware): approve exact production parts
Parts:
- C1: value radial 10 mm -> EEU-FR1A102
- C10, C11, C12, C13, C14, C15, C16, C17, C18, C19, C20, C21, C22, C23, C24, C25, C26, C27, C28, C29, C3, C30, C31, C32, C33, C34, C35, C36, C37, C38, C39, C4, C40, C41, C42, C43, C44, C45, C46, C47, C48, C49, C5, C50, C51, C52, C53, C54, C55, C56, C57, C58, C59, C6, C60, C61, C62, C63, C64, C65, C66, C67, C68, C69, C7, C70, C71, C8, C9: value disc 2.54 mm -> C315C104M5U5TA
- C2: value radial 5 mm -> UVR1C100MDD
- D1: value axial DO-15 -> P6KE6.8A
- F1: value 5x20 mm holder THT -> 3557
- J1: value 2x20 2.54 mm THT -> SSW-120-02-G-D
- J2: value 1x4 2.54 mm THT -> SSW-104-02-G-S
- J3: value 5.5x2.1 mm THT -> PJ-102A
- R1, R2: value axial 1/4 W -> MFR-25FBF52-4K7
- RS1, RS10, RS11, RS12, RS13, RS14, RS15, RS16, RS17, RS18, RS19, RS2, RS20, RS21, RS22, RS23, RS24, RS25, RS26, RS27, RS28, RS29, RS3, RS30, RS31, RS32, RS33, RS34, RS35, RS36, RS37, RS38, RS39, RS4, RS40, RS41, RS42, RS43, RS44, RS45, RS46, RS47, RS48, RS49, RS5, RS50, RS51, RS52, RS53, RS54, RS55, RS56, RS57, RS58, RS59, RS6, RS60, RS61, RS62, RS63, RS64, RS7, RS8, RS9: value axial 14 mm -> KSK-1A66-1015
- SW1, SW10, SW11, SW12, SW2, SW3, SW4, SW5, SW6, SW7, SW8, SW9: value 6x6 mm THT -> B3F-4050
- SW13: value SPST rocker THT -> RA11131100
- TP1, TP2, TP3, TP4: value turret 1.6 mm THT -> 1502-2
- U1, U2, U3, U4: value PDIP-28 -> MCP23017-E/SP
- U10, U11, U12, U13, U14, U15, U16, U17, U18, U19, U20, U21, U22, U23, U24, U25, U26, U27, U28, U29, U30, U31, U32, U33, U34, U35, U36, U37, U38, U39, U40, U41, U42, U43, U44, U45, U46, U47, U48, U49, U50, U51, U52, U53, U54, U55, U56, U57, U58, U59, U6, U60, U61, U62, U63, U64, U65, U66, U67, U68, U69, U7, U8, U9: value PLCC-6 5050 -> SK9822-EC20
- U5: value DIP-14 -> SN74AHCT125N

Commit message: feat(pcb): audit complete fabrication readiness
Parts:
- removed the C10 at (153.0, 355.0)
- removed the C12 at (233.0, 355.0)
- removed the C14 at (313.0, 355.0)
- removed the C16 at (353.0, 315.0)
- removed the C18 at (273.0, 315.0)
- removed the C2 at (84.0, 388.0)
- removed the C21 at (153.0, 315.0)
- removed the C23 at (73.0, 315.0)
- removed the C25 at (113.0, 275.0)
- removed the C27 at (193.0, 275.0)
- removed the C29 at (273.0, 275.0)
- removed the C30 at (313.0, 275.0)
- removed the C32 at (353.0, 235.0)
- removed the C34 at (273.0, 235.0)
- removed the C36 at (193.0, 235.0)
- removed the C38 at (113.0, 235.0)
- removed the C4 at (303.0, 300.0)
- removed the C41 at (113.0, 195.0)
- removed the RS10 at (100.0, 280.0)
- removed the RS24 at (340.0, 320.0)
- removed the RS27 at (300.0, 280.0)
- removed the RS3 at (140.0, 360.0)
- removed the RS42 at (100.0, 120.0)
- removed the RS45 at (60.0, 80.0)
- removed the RS5 at (60.0, 320.0)
- removed the RS52 at (340.0, 200.0)
- removed the RS55 at (300.0, 160.0)
- removed the RS58 at (260.0, 120.0)
- removed the RS60 at (340.0, 120.0)
- removed the RS63 at (300.0, 80.0)
- added C44: C315C104M5U5TA, , F.Cu at (233.0, 195.0)
- added C48: C315C104M5U5TA, , F.Cu at (353.0, 155.0)
- added C5: C315C104M5U5TA, , F.Cu at (143.0, 140.0)
- added C51: C315C104M5U5TA, , F.Cu at (233.0, 155.0)
- added C53: C315C104M5U5TA, , F.Cu at (153.0, 155.0)
- added C55: C315C104M5U5TA, , F.Cu at (73.0, 155.0)
- added C57: C315C104M5U5TA, , F.Cu at (113.0, 115.0)
- added C59: C315C104M5U5TA, , F.Cu at (193.0, 115.0)
- added C60: C315C104M5U5TA, , F.Cu at (233.0, 115.0)
- added C62: C315C104M5U5TA, , F.Cu at (313.0, 115.0)
- added C64: C315C104M5U5TA, , F.Cu at (353.0, 75.0)
- added C66: C315C104M5U5TA, , F.Cu at (273.0, 75.0)
- added C68: C315C104M5U5TA, , F.Cu at (193.0, 75.0)
- added C7: C315C104M5U5TA, , F.Cu at (142.0, 400.0)
- added C71: C315C104M5U5TA, , F.Cu at (73.0, 75.0)
- added C9: C315C104M5U5TA, , F.Cu at (113.0, 355.0)
- added F1: 3557, , F.Cu at (56.0, 413.0)
- added H1: M3 mounting hole, , F.Cu at (80.0, 340.0)
- added H10: M3 mounting hole, , F.Cu at (160.0, 180.0)
- added H11: M3 mounting hole, , F.Cu at (240.0, 180.0)
- added H12: M3 mounting hole, , F.Cu at (320.0, 180.0)
- added H13: M3 mounting hole, , F.Cu at (80.0, 100.0)
- added H14: M3 mounting hole, , F.Cu at (160.0, 100.0)
- added H15: M3 mounting hole, , F.Cu at (240.0, 100.0)
- added H16: M3 mounting hole, , F.Cu at (320.0, 100.0)
- added H17: M3 mounting hole, , F.Cu at (80.0, 400.0)
- added H18: M3 mounting hole, , F.Cu at (160.0, 400.0)
- added H19: M3 mounting hole, , F.Cu at (240.0, 400.0)
- added H2: M3 mounting hole, , F.Cu at (160.0, 340.0)
- added H20: M3 mounting hole, , F.Cu at (320.0, 400.0)
- added H3: M3 mounting hole, , F.Cu at (240.0, 340.0)
- added H4: M3 mounting hole, , F.Cu at (320.0, 340.0)
- added H5: M3 mounting hole, , F.Cu at (80.0, 260.0)
- added H6: M3 mounting hole, , F.Cu at (160.0, 260.0)
- added H7: M3 mounting hole, , F.Cu at (240.0, 260.0)
- added H8: M3 mounting hole, , F.Cu at (320.0, 260.0)
- added H9: M3 mounting hole, , F.Cu at (80.0, 180.0)
- added J3: PJ-102A, , F.Cu at (50.0, 398.0)
- added TP1: 1502-2, , F.Cu at (160.0, 385.0)
- added U22: SK9822-EC20, , F.Cu at (73.0, 267.0)
- added U26: SK9822-EC20, , F.Cu at (233.0, 267.0)
- added U3: MCP23017-E/SP, , F.Cu at (134.0, 140.0)
- added U43: SK9822-EC20, , F.Cu at (273.0, 187.0)
- added U47: SK9822-EC20, , F.Cu at (313.0, 147.0)
- added U52: SK9822-EC20, , F.Cu at (113.0, 147.0)
- added U56: SK9822-EC20, , F.Cu at (153.0, 107.0)
- added U6: SK9822-EC20, , F.Cu at (73.0, 347.0)
- added U63: SK9822-EC20, , F.Cu at (313.0, 67.0)
- added U67: SK9822-EC20, , F.Cu at (153.0, 67.0)
- added U8: SK9822-EC20, , F.Cu at (153.0, 347.0)
- C2: renamed from C3; value C315C104M5U5TA -> UVR1C100MDD
- C42: renamed from F1; value 3557 -> C315C104M5U5TA
- C46: renamed from J3; value PJ-102A -> C315C104M5U5TA
- RS10: renamed from TP1; value 1502-2 -> KSK-1A66-1015
- RS24: renamed from U22; value SK9822-EC20 -> KSK-1A66-1015
- RS27: renamed from U26; value SK9822-EC20 -> KSK-1A66-1015
- RS3: renamed from U3; value MCP23017-E/SP -> KSK-1A66-1015
- RS42: renamed from U43; value SK9822-EC20 -> KSK-1A66-1015
- RS45: renamed from U47; value SK9822-EC20 -> KSK-1A66-1015
- RS5: renamed from U52; value SK9822-EC20 -> KSK-1A66-1015
- RS52: renamed from U56; value SK9822-EC20 -> KSK-1A66-1015
- RS55: renamed from U6; value SK9822-EC20 -> KSK-1A66-1015
- RS58: renamed from U63; value SK9822-EC20 -> KSK-1A66-1015
- RS60: renamed from U67; value SK9822-EC20 -> KSK-1A66-1015
- RS63: renamed from U8; value SK9822-EC20 -> KSK-1A66-1015
- moved C46 332.2 mm to (313.0, 195.0)
- moved RS63 304.8 mm to (300.0, 80.0)
- moved RS55 294.1 mm to (300.0, 160.0)
- moved C32 291.2 mm to (353.0, 235.0)
- moved RS24 272.2 mm to (340.0, 320.0)
- moved RS45 261.7 mm to (60.0, 80.0)
- moved C37 256.1 mm to (153.0, 235.0)
- moved C17 243.3 mm to (313.0, 315.0)
- moved C16 240.0 mm to (353.0, 315.0)
- moved C42 238.6 mm to (153.0, 195.0)
- moved C31 233.2 mm to (353.0, 275.0)
- moved C33 233.2 mm to (313.0, 235.0)
- moved C38 226.3 mm to (113.0, 235.0)
- moved RS3 220.1 mm to (140.0, 360.0)
- moved RS52 208.8 mm to (340.0, 200.0)
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- renumbered C11 to C10, C13 to C11, C15 to C12, C17 to C13, C19 to C14, C20 to C15, C22 to C16, C24 to C17, C26 to C18, C28 to C19, C31 to C20, C33 to C21, C35 to C22, C37 to C23, C39 to C24, C40 to C25, C42 to C26, C44 to C27, C46 to C28, C48 to C29, C5 to C3, C51 to C30, C53 to C31, C55 to C32, C57 to C33, C59 to C34, C60 to C35, C62 to C36, C64 to C37, C66 to C38, C68 to C39, C7 to C4, C71 to C40, C9 to C41
Connections:
- C2 pad 1: +3V3 -> +5V
- C4 pad 1: +5V -> +3V3
- C42 pad 1: DC_IN -> +5V
- C42 pad 2: DC_FUSED -> GND
- C46 pad 1: DC_IN -> +5V
- RS10 pad 1: +5V -> SQ_B3
- RS24 pad 1: +5V -> SQ_H2
- RS27 pad 1: +5V -> SQ_G3
- RS3 pad 1: SQ_A7 -> SQ_C1
- RS3 pad 2: SQ_B7 -> GND
- RS42 pad 1: +5V -> SQ_B7
- RS45 pad 1: +5V -> SQ_A8
- RS5 pad 1: +5V -> SQ_A2
- RS52 pad 1: +5V -> SQ_H5
- RS55 pad 1: +5V -> SQ_G6
- RS58 pad 1: +5V -> SQ_F7
- RS60 pad 1: +5V -> SQ_H7
- RS63 pad 1: +5V -> SQ_G8
Routing:
- net LED_D8: track 42.4 -> 40.4 mm
- net LED_D56: track 42.4 -> 40.4 mm
- net LED_D48: track 55.6 -> 53.6 mm
- net LED_D40: track 42.4 -> 40.4 mm
- net LED_D32: track 55.6 -> 53.6 mm
- net LED_D24: track 42.4 -> 40.4 mm
- net LED_D16: track 55.6 -> 53.6 mm

Commit message: feat(pcb): route sensor grid and control signals
Routing:
- net LED_CLK_5V: track 0.00 -> 188.1 mm
- net BTN_RESET: track 0.00 -> 175.1 mm, vias 0 -> 3
- net N$205: track 0.00 -> 169.4 mm, vias 0 -> 4
- net N$138: track 0.00 -> 169.4 mm, vias 0 -> 4
- net LED_DATA_5V: track 0.00 -> 168.1 mm, vias 0 -> 3
- net BTN_F5: track 0.00 -> 161.7 mm, vias 0 -> 1
- net SQ_H8: track 0.00 -> 160.9 mm, vias 0 -> 3
- net SQ_H4: track 0.00 -> 160.9 mm, vias 0 -> 3
- net SQ_E5: track 0.00 -> 145.9 mm
- net SQ_A5: track 0.00 -> 145.9 mm
- net SQ_E1: track 0.00 -> 145.9 mm
- net SQ_A1: track 0.00 -> 145.9 mm
- net BTN_F4: track 0.00 -> 144.1 mm, vias 0 -> 2
- net SPI_CLK_3V3: track 0.00 -> 143.5 mm, vias 0 -> 1
- net SQ_A8: track 0.00 -> 139.9 mm
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- added copper zone on B.Cu, net +3V3
- added copper zone on F.Cu, net +3V3
