File: hardware/pcb/chess-board.kicad_pcb (KiCad board)
At the start: 4 copper layers, 320 x 360 mm, 248 parts, among them J1 SSW-120-02-G-D, J2 SSW-104-02-G-S, J3 PJ-102A, SW1 B3F-4050, SW10 B3F-4050, SW11 B3F-4050, SW12 B3F-4050, SW13 RA11131100, SW2 B3F-4050, SW3 B3F-4050, SW4 B3F-4050, SW5 B3F-4050, SW6 B3F-4050, SW7 B3F-4050, SW8 B3F-4050, SW9 B3F-4050, U1 MCP23017-E/SP, U10 SK9822-EC20, U11 SK9822-EC20, U12 SK9822-EC20, U13 SK9822-EC20, U14 SK9822-EC20, U15 SK9822-EC20, U16 SK9822-EC20, U17 SK9822-EC20, U18 SK9822-EC20, U19 SK9822-EC20, U2 MCP23017-E/SP, U20 SK9822-EC20, U21 SK9822-EC20, U22 SK9822-EC20, U23 SK9822-EC20, U24 SK9822-EC20, U25 SK9822-EC20, U26 SK9822-EC20, U27 SK9822-EC20, U28 SK9822-EC20, U29 SK9822-EC20, U3 MCP23017-E/SP, U30 SK9822-EC20, U31 SK9822-EC20, U32 SK9822-EC20, U33 SK9822-EC20, U34 SK9822-EC20, U35 SK9822-EC20, U36 SK9822-EC20, U37 SK9822-EC20, U38 SK9822-EC20, U39 SK9822-EC20, U4 MCP23017-E/SP, U40 SK9822-EC20, U41 SK9822-EC20, U42 SK9822-EC20, U43 SK9822-EC20, U44 SK9822-EC20, U45 SK9822-EC20, U46 SK9822-EC20, U47 SK9822-EC20, U48 SK9822-EC20, U49 SK9822-EC20, U5 SN74AHCT125N, U50 SK9822-EC20, U51 SK9822-EC20, U52 SK9822-EC20, U53 SK9822-EC20, U54 SK9822-EC20, U55 SK9822-EC20, U56 SK9822-EC20, U57 SK9822-EC20, U58 SK9822-EC20, U59 SK9822-EC20, U6 SK9822-EC20, U60 SK9822-EC20, U61 SK9822-EC20, U62 SK9822-EC20, U63 SK9822-EC20, U64 SK9822-EC20, U65 SK9822-EC20, U66 SK9822-EC20, U67 SK9822-EC20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

Commit message: feat(pcb): complete routed native KiCad project
Connections:
- J1 pad 10: N$105 -> unconnected-(J1-Pad10)
- J1 pad 12: N$106 -> unconnected-(J1-Pad12)
- J1 pad 13: N$107 -> unconnected-(J1-Pad13)
- J1 pad 21: N$108 -> unconnected-(J1-Pad21)
- J1 pad 22: N$109 -> unconnected-(J1-Pad22)
- J1 pad 24: N$110 -> unconnected-(J1-Pad24)
- J1 pad 26: N$111 -> unconnected-(J1-Pad26)
- J1 pad 27: N$112 -> unconnected-(J1-Pad27)
- J1 pad 28: N$113 -> unconnected-(J1-Pad28)
- J1 pad 37: N$114 -> unconnected-(J1-Pad37)
- J1 pad 8: N$115 -> unconnected-(J1-Pad8)
- U1 pad 11: N$116 -> unconnected-(U1-Pad11)
- U1 pad 14: N$117 -> unconnected-(U1-Pad14)
- U1 pad 19: N$118 -> unconnected-(U1-Pad19)
- U2 pad 11: N$139 -> unconnected-(U2-Pad11)
- U2 pad 14: N$140 -> unconnected-(U2-Pad14)
- U2 pad 19: N$141 -> unconnected-(U2-Pad19)
- U3 pad 11: N$158 -> unconnected-(U3-Pad11)
- U3 pad 14: N$159 -> unconnected-(U3-Pad14)
- U3 pad 19: N$160 -> unconnected-(U3-Pad19)
- U4 pad 11: N$179 -> unconnected-(U4-Pad11)
- U4 pad 14: N$180 -> unconnected-(U4-Pad14)
- U4 pad 19: N$181 -> unconnected-(U4-Pad19)
- U5 pad 11: N$200 -> unconnected-(U5-Pad11)
- U5 pad 8: N$201 -> unconnected-(U5-Pad8)
- U69 pad 5: LED_DATA_LAST -> unconnected-(U69-Pad5)
- U69 pad 6: LED_CLK_LAST -> unconnected-(U69-Pad6)
Routing:
- net I2C_SCL: track 0.00 -> 725.3 mm
- net I2C_SDA: track 0.00 -> 707.2 mm
- net SENSE_IRQ: track 0.00 -> 596.1 mm
- net BTN_F3: track 4.50 -> 91.5 mm
- net BTN_F1: track 4.50 -> 88.5 mm
- net BTN_OK: track 4.50 -> 83.9 mm
- net BTN_LEFT: track 4.50 -> 81.9 mm
- net BTN_RIGHT: track 4.50 -> 76.2 mm
- net N$205: track 169.4 -> 104.4 mm
- net N$138: track 169.4 -> 104.4 mm
- net SQ_H8: track 160.9 -> 102.9 mm, vias 3 -> 0
- net SQ_H4: track 160.9 -> 102.9 mm, vias 3 -> 0
- net SQ_C2: track 41.3 -> 92.3 mm, vias 0 -> 1
- net SQ_C6: track 41.3 -> 92.3 mm, vias 0 -> 1
- net BTN_DOWN: track 4.50 -> 54.1 mm
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- added copper zone on In3.Cu, net +3V3
- removed copper zone on B.Cu, net +3V3
- removed copper zone on F.Cu, net +3V3
Other:
- copper layers 4 -> 8

Commit message: fix(pcb): correct reviewed component pinouts
Connections:
- U10 pad 1: +5V -> N$119
- U10 pad 2: GND -> N$120
- U10 pad 3: N$119 -> GND
- U10 pad 4: N$120 -> +5V
- U10 pad 5: N$121 -> N$122
- U10 pad 6: N$122 -> N$121
- U11 pad 1: +5V -> N$121
- U11 pad 2: GND -> N$122
- U11 pad 3: N$121 -> GND
- U11 pad 4: N$122 -> +5V
- U11 pad 5: N$123 -> N$124
- U11 pad 6: N$124 -> N$123
- U12 pad 1: +5V -> N$123
- U12 pad 2: GND -> N$124
- U12 pad 3: N$123 -> GND
- U12 pad 4: N$124 -> +5V
- U12 pad 5: N$125 -> N$126
- U12 pad 6: N$126 -> N$125
- U13 pad 1: +5V -> N$125
- U13 pad 2: GND -> N$126
- U13 pad 3: N$125 -> GND
- U13 pad 4: N$126 -> +5V
- U13 pad 5: LED_D8 -> LED_C8
- U13 pad 6: LED_C8 -> LED_D8
- U14 pad 1: +5V -> LED_D8
- U14 pad 2: GND -> LED_C8
- U14 pad 3: LED_D8 -> GND
- U14 pad 4: LED_C8 -> +5V
- U14 pad 5: N$127 -> N$128
- U14 pad 6: N$128 -> N$127
- U15 pad 1: +5V -> N$127
- U15 pad 2: GND -> N$128
- U15 pad 3: N$127 -> GND
- U15 pad 4: N$128 -> +5V
- U15 pad 5: N$129 -> N$130
- U15 pad 6: N$130 -> N$129
- U16 pad 1: +5V -> N$129
- U16 pad 2: GND -> N$130
- U16 pad 3: N$129 -> GND
- U16 pad 4: N$130 -> +5V
- U16 pad 5: N$131 -> N$132
- U16 pad 6: N$132 -> N$131
- U17 pad 1: +5V -> N$131
- U17 pad 2: GND -> N$132
- U17 pad 3: N$131 -> GND
- U17 pad 4: N$132 -> +5V
- U17 pad 5: N$133 -> N$134
- U17 pad 6: N$134 -> N$133
- U18 pad 1: +5V -> N$133
- U18 pad 2: GND -> N$134
- U18 pad 3: N$133 -> GND
- U18 pad 4: N$134 -> +5V
- U18 pad 5: N$135 -> N$136
- U18 pad 6: N$136 -> N$135
- U19 pad 1: +5V -> N$135
- U19 pad 2: GND -> N$136
- U19 pad 3: N$135 -> GND
- U19 pad 4: N$136 -> +5V
- U19 pad 5: N$137 -> N$138
- U19 pad 6: N$138 -> N$137
- U20 pad 1: +5V -> N$137
- U20 pad 2: GND -> N$138
- U20 pad 3: N$137 -> GND
- U20 pad 4: N$138 -> +5V
- U20 pad 5: N$142 -> N$143
- U20 pad 6: N$143 -> N$142
- U21 pad 1: +5V -> N$142
- U21 pad 2: GND -> N$143
- U21 pad 3: N$142 -> GND
- U21 pad 4: N$143 -> +5V
- U21 pad 5: LED_D16 -> LED_C16
- U21 pad 6: LED_C16 -> LED_D16
- U22 pad 1: +5V -> LED_D16
- U22 pad 2: GND -> LED_C16
- U22 pad 3: LED_D16 -> GND
- U22 pad 4: LED_C16 -> +5V
- U22 pad 5: N$144 -> N$145
- U22 pad 6: N$145 -> N$144
- U23 pad 1: +5V -> N$144
- U23 pad 2: GND -> N$145
- U23 pad 3: N$144 -> GND
- U23 pad 4: N$145 -> +5V
- U23 pad 5: N$146 -> N$147
- U23 pad 6: N$147 -> N$146
- U24 pad 1: +5V -> N$146
- U24 pad 2: GND -> N$147
- U24 pad 3: N$146 -> GND
- U24 pad 4: N$147 -> +5V
- U24 pad 5: N$148 -> N$149
- U24 pad 6: N$149 -> N$148
- U25 pad 1: +5V -> N$148
- U25 pad 2: GND -> N$149
- U25 pad 3: N$148 -> GND
- U25 pad 4: N$149 -> +5V
- U25 pad 5: N$150 -> N$151
- U25 pad 6: N$151 -> N$150
- U26 pad 1: +5V -> N$150
- U26 pad 2: GND -> N$151
- U26 pad 3: N$150 -> GND
- U26 pad 4: N$151 -> +5V
- U26 pad 5: N$152 -> N$153
- U26 pad 6: N$153 -> N$152
- U27 pad 1: +5V -> N$152
- U27 pad 2: GND -> N$153
- U27 pad 3: N$152 -> GND
- U27 pad 4: N$153 -> +5V
- U27 pad 5: N$154 -> N$155
- U27 pad 6: N$155 -> N$154
- U28 pad 1: +5V -> N$154
- U28 pad 2: GND -> N$155
- U28 pad 3: N$154 -> GND
- U28 pad 4: N$155 -> +5V
- U28 pad 5: N$156 -> N$157
- U28 pad 6: N$157 -> N$156
- U29 pad 1: +5V -> N$156
- U29 pad 2: GND -> N$157
- U29 pad 3: N$156 -> GND
- U29 pad 4: N$157 -> +5V
- U29 pad 5: LED_D24 -> LED_C24
- U29 pad 6: LED_C24 -> LED_D24
- U30 pad 1: +5V -> LED_D24
- U30 pad 2: GND -> LED_C24
- U30 pad 3: LED_D24 -> GND
- U30 pad 4: LED_C24 -> +5V
- U30 pad 5: N$161 -> N$162
- U30 pad 6: N$162 -> N$161
- U31 pad 1: +5V -> N$161
- U31 pad 2: GND -> N$162
- U31 pad 3: N$161 -> GND
- U31 pad 4: N$162 -> +5V
- U31 pad 5: N$163 -> N$164
- U31 pad 6: N$164 -> N$163
- U32 pad 1: +5V -> N$163
- U32 pad 2: GND -> N$164
- U32 pad 3: N$163 -> GND
- U32 pad 4: N$164 -> +5V
- U32 pad 5: N$165 -> N$166
- U32 pad 6: N$166 -> N$165
- U33 pad 1: +5V -> N$165
- U33 pad 2: GND -> N$166
- U33 pad 3: N$165 -> GND
- U33 pad 4: N$166 -> +5V
- U33 pad 5: N$167 -> N$168
- U33 pad 6: N$168 -> N$167
- U34 pad 1: +5V -> N$167
- U34 pad 2: GND -> N$168
- U34 pad 3: N$167 -> GND
- U34 pad 4: N$168 -> +5V
- U34 pad 5: N$169 -> N$170
- U34 pad 6: N$170 -> N$169
- U35 pad 1: +5V -> N$169
- U35 pad 2: GND -> N$170
- U35 pad 3: N$169 -> GND
- U35 pad 4: N$170 -> +5V
- U35 pad 5: N$171 -> N$172
- U35 pad 6: N$172 -> N$171
- U36 pad 1: +5V -> N$171
- U36 pad 2: GND -> N$172
- U36 pad 3: N$171 -> GND
- U36 pad 4: N$172 -> +5V
- U36 pad 5: N$173 -> N$174
- U36 pad 6: N$174 -> N$173
- U37 pad 1: +5V -> N$173
- U37 pad 2: GND -> N$174
- U37 pad 3: N$173 -> GND
- U37 pad 4: N$174 -> +5V
- U37 pad 5: LED_D32 -> LED_C32
- U37 pad 6: LED_C32 -> LED_D32
- U38 pad 1: +5V -> LED_D32
- U38 pad 2: GND -> LED_C32
- U38 pad 3: LED_D32 -> GND
- U38 pad 4: LED_C32 -> +5V
- U38 pad 5: N$175 -> N$176
- U38 pad 6: N$176 -> N$175
- U39 pad 1: +5V -> N$175
- U39 pad 2: GND -> N$176
- U39 pad 3: N$175 -> GND
- U39 pad 4: N$176 -> +5V
- U39 pad 5: N$177 -> N$178
- U39 pad 6: N$178 -> N$177
- U40 pad 1: +5V -> N$177
- U40 pad 2: GND -> N$178
- U40 pad 3: N$177 -> GND
- U40 pad 4: N$178 -> +5V
- U40 pad 5: N$182 -> N$183
- U40 pad 6: N$183 -> N$182
- U41 pad 1: +5V -> N$182
- U41 pad 2: GND -> N$183
- U41 pad 3: N$182 -> GND
- U41 pad 4: N$183 -> +5V
- U41 pad 5: N$184 -> N$185
- U41 pad 6: N$185 -> N$184
- U42 pad 1: +5V -> N$184
- U42 pad 2: GND -> N$185
- U42 pad 3: N$184 -> GND
- U42 pad 4: N$185 -> +5V
- U42 pad 5: N$186 -> N$187
- U42 pad 6: N$187 -> N$186
- U43 pad 1: +5V -> N$186
- U43 pad 2: GND -> N$187
- U43 pad 3: N$186 -> GND
- U43 pad 4: N$187 -> +5V
- U43 pad 5: N$188 -> N$189
- U43 pad 6: N$189 -> N$188
- U44 pad 1: +5V -> N$188
- U44 pad 2: GND -> N$189
- U44 pad 3: N$188 -> GND
- U44 pad 4: N$189 -> +5V
- U44 pad 5: N$190 -> N$191
- U44 pad 6: N$191 -> N$190
- U45 pad 1: +5V -> N$190
- U45 pad 2: GND -> N$191
- U45 pad 3: N$190 -> GND
- U45 pad 4: N$191 -> +5V
- U45 pad 5: LED_D40 -> LED_C40
- U45 pad 6: LED_C40 -> LED_D40
- U46 pad 1: +5V -> LED_D40
- U46 pad 2: GND -> LED_C40
- U46 pad 3: LED_D40 -> GND
- U46 pad 4: LED_C40 -> +5V
- U46 pad 5: N$192 -> N$193
- U46 pad 6: N$193 -> N$192
- U47 pad 1: +5V -> N$192
- U47 pad 2: GND -> N$193
- U47 pad 3: N$192 -> GND
- U47 pad 4: N$193 -> +5V
- U47 pad 5: N$194 -> N$195
- U47 pad 6: N$195 -> N$194
- U48 pad 1: +5V -> N$194
- U48 pad 2: GND -> N$195
- U48 pad 3: N$194 -> GND
- U48 pad 4: N$195 -> +5V
- U48 pad 5: N$196 -> N$197
- U48 pad 6: N$197 -> N$196
- U49 pad 1: +5V -> N$196
- U49 pad 2: GND -> N$197
- U49 pad 3: N$196 -> GND
- U49 pad 4: N$197 -> +5V
- U49 pad 5: N$198 -> N$199
- U49 pad 6: N$199 -> N$198
- U50 pad 1: +5V -> N$198
- U50 pad 2: GND -> N$199
- U50 pad 3: N$198 -> GND
- U50 pad 4: N$199 -> +5V
- U50 pad 5: N$202 -> N$203
- U50 pad 6: N$203 -> N$202
- U51 pad 1: +5V -> N$202
- U51 pad 2: GND -> N$203
- U51 pad 3: N$202 -> GND
- U51 pad 4: N$203 -> +5V
- U51 pad 5: N$204 -> N$205
- U51 pad 6: N$205 -> N$204
- U52 pad 1: +5V -> N$204
- U52 pad 2: GND -> N$205
- U52 pad 3: N$204 -> GND
- U52 pad 4: N$205 -> +5V
- U52 pad 5: N$206 -> N$207
- U52 pad 6: N$207 -> N$206
- U53 pad 1: +5V -> N$206
- U53 pad 2: GND -> N$207
- U53 pad 3: N$206 -> GND
- U53 pad 4: N$207 -> +5V
- U53 pad 5: LED_D48 -> LED_C48
- U53 pad 6: LED_C48 -> LED_D48
- U54 pad 1: +5V -> LED_D48
- U54 pad 2: GND -> LED_C48
- U54 pad 3: LED_D48 -> GND
- U54 pad 4: LED_C48 -> +5V
- U54 pad 5: N$208 -> N$209
- U54 pad 6: N$209 -> N$208
- U55 pad 1: +5V -> N$208
- U55 pad 2: GND -> N$209
- U55 pad 3: N$208 -> GND
- U55 pad 4: N$209 -> +5V
- U55 pad 5: N$210 -> N$211
- U55 pad 6: N$211 -> N$210
- U56 pad 1: +5V -> N$210
- U56 pad 2: GND -> N$211
- U56 pad 3: N$210 -> GND
- U56 pad 4: N$211 -> +5V
- U56 pad 5: N$212 -> N$213
- U56 pad 6: N$213 -> N$212
- U57 pad 1: +5V -> N$212
- U57 pad 2: GND -> N$213
- U57 pad 3: N$212 -> GND
- U57 pad 4: N$213 -> +5V
- U57 pad 5: N$214 -> N$215
- U57 pad 6: N$215 -> N$214
- U58 pad 1: +5V -> N$214
- U58 pad 2: GND -> N$215
- U58 pad 3: N$214 -> GND
- U58 pad 4: N$215 -> +5V
- U58 pad 5: N$216 -> N$217
- U58 pad 6: N$217 -> N$216
- U59 pad 1: +5V -> N$216
- U59 pad 2: GND -> N$217
- U59 pad 3: N$216 -> GND
- U59 pad 4: N$217 -> +5V
- U59 pad 5: N$218 -> N$219
- U59 pad 6: N$219 -> N$218
- U6 pad 1: +5V -> LED_DATA_5V
- U6 pad 2: GND -> LED_CLK_5V
- U6 pad 3: LED_DATA_5V -> GND
- U6 pad 4: LED_CLK_5V -> +5V
- U6 pad 5: N$220 -> N$221
- U6 pad 6: N$221 -> N$220
- U60 pad 1: +5V -> N$218
- U60 pad 2: GND -> N$219
- U60 pad 3: N$218 -> GND
- U60 pad 4: N$219 -> +5V
- U60 pad 5: N$222 -> N$223
- U60 pad 6: N$223 -> N$222
- U61 pad 1: +5V -> N$222
- U61 pad 2: GND -> N$223
- U61 pad 3: N$222 -> GND
- U61 pad 4: N$223 -> +5V
- U61 pad 5: LED_D56 -> LED_C56
- U61 pad 6: LED_C56 -> LED_D56
- U62 pad 1: +5V -> LED_D56
- U62 pad 2: GND -> LED_C56
- U62 pad 3: LED_D56 -> GND
- U62 pad 4: LED_C56 -> +5V
- U62 pad 5: N$224 -> N$225
- U62 pad 6: N$225 -> N$224
- U63 pad 1: +5V -> N$224
- U63 pad 2: GND -> N$225
- U63 pad 3: N$224 -> GND
- U63 pad 4: N$225 -> +5V
- U63 pad 5: N$226 -> N$227
- U63 pad 6: N$227 -> N$226
- U64 pad 1: +5V -> N$226
- U64 pad 2: GND -> N$227
- U64 pad 3: N$226 -> GND
- U64 pad 4: N$227 -> +5V
- U64 pad 5: N$228 -> N$229
- U64 pad 6: N$229 -> N$228
- U65 pad 1: +5V -> N$228
- U65 pad 2: GND -> N$229
- U65 pad 3: N$228 -> GND
- U65 pad 4: N$229 -> +5V
- U65 pad 5: N$230 -> N$231
- U65 pad 6: N$231 -> N$230
- U66 pad 1: +5V -> N$230
- U66 pad 2: GND -> N$231
- U66 pad 3: N$230 -> GND
- U66 pad 4: N$231 -> +5V
- U66 pad 5: N$232 -> N$233
- U66 pad 6: N$233 -> N$232
- U67 pad 1: +5V -> N$232
- U67 pad 2: GND -> N$233
- U67 pad 3: N$232 -> GND
- U67 pad 4: N$233 -> +5V
- U67 pad 5: N$234 -> N$235
- U67 pad 6: N$235 -> N$234
- U68 pad 1: +5V -> N$234
- U68 pad 2: GND -> N$235
- U68 pad 3: N$234 -> GND
- U68 pad 4: N$235 -> +5V
- U68 pad 5: N$236 -> N$237
- U68 pad 6: N$237 -> N$236
- U69 pad 1: +5V -> N$236
- U69 pad 2: GND -> N$237
- U69 pad 3: N$236 -> GND
- U69 pad 4: N$237 -> +5V
- U7 pad 1: +5V -> N$220
- U7 pad 2: GND -> N$221
- U7 pad 3: N$220 -> GND
- U7 pad 4: N$221 -> +5V
- U7 pad 5: N$238 -> N$239
- U7 pad 6: N$239 -> N$238
- U8 pad 1: +5V -> N$238
- U8 pad 2: GND -> N$239
- U8 pad 3: N$238 -> GND
- U8 pad 4: N$239 -> +5V
- U8 pad 5: N$240 -> N$241
- U8 pad 6: N$241 -> N$240
- U9 pad 1: +5V -> N$240
- U9 pad 2: GND -> N$241
- U9 pad 3: N$240 -> GND
- U9 pad 4: N$241 -> +5V
- U9 pad 5: N$119 -> N$120
- U9 pad 6: N$120 -> N$119
