File: hardware/pcb/chess-board.kicad_sch (KiCad schematic)
At the start: 228 parts, among them J1 SSW-120-02-G-D, J2 SSW-104-02-G-S, J3 PJ-102A, SW1 B3F-4050, SW10 B3F-4050, SW11 B3F-4050, SW12 B3F-4050, SW13 RA11131100, SW2 B3F-4050, SW3 B3F-4050, SW4 B3F-4050, SW5 B3F-4050, SW6 B3F-4050, SW7 B3F-4050, SW8 B3F-4050, SW9 B3F-4050, U1 MCP23017-E/SP, U10 SK9822-EC20, U11 SK9822-EC20, U12 SK9822-EC20, U13 SK9822-EC20, U14 SK9822-EC20, U15 SK9822-EC20, U16 SK9822-EC20, U17 SK9822-EC20, U18 SK9822-EC20, U19 SK9822-EC20, U2 MCP23017-E/SP, U20 SK9822-EC20, U21 SK9822-EC20, U22 SK9822-EC20, U23 SK9822-EC20, U24 SK9822-EC20, U25 SK9822-EC20, U26 SK9822-EC20, U27 SK9822-EC20, U28 SK9822-EC20, U29 SK9822-EC20, U3 MCP23017-E/SP, U30 SK9822-EC20, U31 SK9822-EC20, U32 SK9822-EC20, U33 SK9822-EC20, U34 SK9822-EC20, U35 SK9822-EC20, U36 SK9822-EC20, U37 SK9822-EC20, U38 SK9822-EC20, U39 SK9822-EC20, U4 MCP23017-E/SP, U40 SK9822-EC20, U41 SK9822-EC20, U42 SK9822-EC20, U43 SK9822-EC20, U44 SK9822-EC20, U45 SK9822-EC20, U46 SK9822-EC20, U47 SK9822-EC20, U48 SK9822-EC20, U49 SK9822-EC20, U5 SN74AHCT125N, U50 SK9822-EC20, U51 SK9822-EC20, U52 SK9822-EC20, U53 SK9822-EC20, U54 SK9822-EC20, U55 SK9822-EC20, U56 SK9822-EC20, U57 SK9822-EC20, U58 SK9822-EC20, U59 SK9822-EC20, U6 SK9822-EC20, U60 SK9822-EC20, U61 SK9822-EC20, U62 SK9822-EC20, U63 SK9822-EC20, U64 SK9822-EC20, U65 SK9822-EC20, U66 SK9822-EC20, U67 SK9822-EC20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

Commit message: fix(pcb): correct reviewed component pinouts
Connections:
- net +5V: now also U10.4, U11.4, U12.4, U13.4, U14.4, U15.4, U16.4, U17.4, U18.4, U19.4, U20.4, U21.4, U22.4, U23.4, U24.4, U25.4, U26.4, U27.4, U28.4, U29.4, U30.4, U31.4, U32.4, U33.4, U34.4, U35.4, U36.4, U37.4, U38.4, U39.4, U40.4, U41.4, U42.4, U43.4, U44.4, U45.4, U46.4, U47.4, U48.4, U49.4, U50.4, U51.4, U52.4, U53.4, U54.4, U55.4, U56.4, U57.4, U58.4, U59.4, U6.4, U60.4, U61.4, U62.4, U63.4, U64.4, U65.4, U66.4, U67.4, U68.4, U69.4, U7.4, U8.4, U9.4; no longer U10.1, U11.1, U12.1, U13.1, U14.1, U15.1, U16.1, U17.1, U18.1, U19.1, U20.1, U21.1, U22.1, U23.1, U24.1, U25.1, U26.1, U27.1, U28.1, U29.1, U30.1, U31.1, U32.1, U33.1, U34.1, U35.1, U36.1, U37.1, U38.1, U39.1, U40.1, U41.1, U42.1, U43.1, U44.1, U45.1, U46.1, U47.1, U48.1, U49.1, U50.1, U51.1, U52.1, U53.1, U54.1, U55.1, U56.1, U57.1, U58.1, U59.1, U6.1, U60.1, U61.1, U62.1, U63.1, U64.1, U65.1, U66.1, U67.1, U68.1, U69.1, U7.1, U8.1, U9.1
- net GND: now also J3.3, U10.3, U11.3, U12.3, U13.3, U14.3, U15.3, U16.3, U17.3, U18.3, U19.3, U20.3, U21.3, U22.3, U23.3, U24.3, U25.3, U26.3, U27.3, U28.3, U29.3, U30.3, U31.3, U32.3, U33.3, U34.3, U35.3, U36.3, U37.3, U38.3, U39.3, U40.3, U41.3, U42.3, U43.3, U44.3, U45.3, U46.3, U47.3, U48.3, U49.3, U50.3, U51.3, U52.3, U53.3, U54.3, U55.3, U56.3, U57.3, U58.3, U59.3, U6.3, U60.3, U61.3, U62.3, U63.3, U64.3, U65.3, U66.3, U67.3, U68.3, U69.3, U7.3, U8.3, U9.3; no longer J3.2b, U10.2, U11.2, U12.2, U13.2, U14.2, U15.2, U16.2, U17.2, U18.2, U19.2, U20.2, U21.2, U22.2, U23.2, U24.2, U25.2, U26.2, U27.2, U28.2, U29.2, U30.2, U31.2, U32.2, U33.2, U34.2, U35.2, U36.2, U37.2, U38.2, U39.2, U40.2, U41.2, U42.2, U43.2, U44.2, U45.2, U46.2, U47.2, U48.2, U49.2, U50.2, U51.2, U52.2, U53.2, U54.2, U55.2, U56.2, U57.2, U58.2, U59.2, U6.2, U60.2, U61.2, U62.2, U63.2, U64.2, U65.2, U66.2, U67.2, U68.2, U69.2, U7.2, U8.2, U9.2
- net LED_C16: now also U21.5, U22.2; no longer U21.6, U22.4
- net LED_C24: now also U29.5, U30.2; no longer U29.6, U30.4
- net LED_C32: now also U37.5, U38.2; no longer U37.6, U38.4
- net LED_C40: now also U45.5, U46.2; no longer U45.6, U46.4
- net LED_C48: now also U53.5, U54.2; no longer U53.6, U54.4
- net LED_C56: now also U61.5, U62.2; no longer U61.6, U62.4
- net LED_C8: now also U13.5, U14.2; no longer U13.6, U14.4
- net LED_CLK_5V: now also U6.2; no longer U6.4
- net LED_D16: now also U21.6, U22.1; no longer U21.5, U22.3
- net LED_D24: now also U29.6, U30.1; no longer U29.5, U30.3
- net LED_D32: now also U37.6, U38.1; no longer U37.5, U38.3
- net LED_D40: now also U45.6, U46.1; no longer U45.5, U46.3
- net LED_D48: now also U53.6, U54.1; no longer U53.5, U54.3
- net LED_D56: now also U61.6, U62.1; no longer U61.5, U62.3
- net LED_D8: now also U13.6, U14.1; no longer U13.5, U14.3
- net LED_DATA_5V: now also U6.1; no longer U6.3
- net N$119: now also U10.1, U9.6; no longer U10.3, U9.5
- net N$120: now also U10.2, U9.5; no longer U10.4, U9.6
- net N$121: now also U10.6, U11.1; no longer U10.5, U11.3
- net N$122: now also U10.5, U11.2; no longer U10.6, U11.4
- net N$123: now also U11.6, U12.1; no longer U11.5, U12.3
- net N$124: now also U11.5, U12.2; no longer U11.6, U12.4
- net N$125: now also U12.6, U13.1; no longer U12.5, U13.3
- net N$126: now also U12.5, U13.2; no longer U12.6, U13.4
- net N$127: now also U14.6, U15.1; no longer U14.5, U15.3
- net N$128: now also U14.5, U15.2; no longer U14.6, U15.4
- net N$129: now also U15.6, U16.1; no longer U15.5, U16.3
- net N$130: now also U15.5, U16.2; no longer U15.6, U16.4
- net N$131: now also U16.6, U17.1; no longer U16.5, U17.3
- net N$132: now also U16.5, U17.2; no longer U16.6, U17.4
- net N$133: now also U17.6, U18.1; no longer U17.5, U18.3
- net N$134: now also U17.5, U18.2; no longer U17.6, U18.4
- net N$135: now also U18.6, U19.1; no longer U18.5, U19.3
- net N$136: now also U18.5, U19.2; no longer U18.6, U19.4
- net N$137: now also U19.6, U20.1; no longer U19.5, U20.3
- net N$138: now also U19.5, U20.2; no longer U19.6, U20.4
- net N$142: now also U20.6, U21.1; no longer U20.5, U21.3
- net N$143: now also U20.5, U21.2; no longer U20.6, U21.4
- net N$144: now also U22.6, U23.1; no longer U22.5, U23.3
- net N$145: now also U22.5, U23.2; no longer U22.6, U23.4
- net N$146: now also U23.6, U24.1; no longer U23.5, U24.3
- net N$147: now also U23.5, U24.2; no longer U23.6, U24.4
- net N$148: now also U24.6, U25.1; no longer U24.5, U25.3
- net N$149: now also U24.5, U25.2; no longer U24.6, U25.4
- net N$150: now also U25.6, U26.1; no longer U25.5, U26.3
- net N$151: now also U25.5, U26.2; no longer U25.6, U26.4
- net N$152: now also U26.6, U27.1; no longer U26.5, U27.3
- net N$153: now also U26.5, U27.2; no longer U26.6, U27.4
- net N$154: now also U27.6, U28.1; no longer U27.5, U28.3
- net N$155: now also U27.5, U28.2; no longer U27.6, U28.4
- net N$156: now also U28.6, U29.1; no longer U28.5, U29.3
- net N$157: now also U28.5, U29.2; no longer U28.6, U29.4
- net N$161: now also U30.6, U31.1; no longer U30.5, U31.3
- net N$162: now also U30.5, U31.2; no longer U30.6, U31.4
- net N$163: now also U31.6, U32.1; no longer U31.5, U32.3
- net N$164: now also U31.5, U32.2; no longer U31.6, U32.4
- net N$165: now also U32.6, U33.1; no longer U32.5, U33.3
- net N$166: now also U32.5, U33.2; no longer U32.6, U33.4
- net N$167: now also U33.6, U34.1; no longer U33.5, U34.3
- net N$168: now also U33.5, U34.2; no longer U33.6, U34.4
- net N$169: now also U34.6, U35.1; no longer U34.5, U35.3
- net N$170: now also U34.5, U35.2; no longer U34.6, U35.4
- net N$171: now also U35.6, U36.1; no longer U35.5, U36.3
- net N$172: now also U35.5, U36.2; no longer U35.6, U36.4
- net N$173: now also U36.6, U37.1; no longer U36.5, U37.3
- net N$174: now also U36.5, U37.2; no longer U36.6, U37.4
- net N$175: now also U38.6, U39.1; no longer U38.5, U39.3
- net N$176: now also U38.5, U39.2; no longer U38.6, U39.4
- net N$177: now also U39.6, U40.1; no longer U39.5, U40.3
- net N$178: now also U39.5, U40.2; no longer U39.6, U40.4
- net N$182: now also U40.6, U41.1; no longer U40.5, U41.3
- net N$183: now also U40.5, U41.2; no longer U40.6, U41.4
- net N$184: now also U41.6, U42.1; no longer U41.5, U42.3
- net N$185: now also U41.5, U42.2; no longer U41.6, U42.4
- net N$186: now also U42.6, U43.1; no longer U42.5, U43.3
- net N$187: now also U42.5, U43.2; no longer U42.6, U43.4
- net N$188: now also U43.6, U44.1; no longer U43.5, U44.3
- net N$189: now also U43.5, U44.2; no longer U43.6, U44.4
- net N$190: now also U44.6, U45.1; no longer U44.5, U45.3
- net N$191: now also U44.5, U45.2; no longer U44.6, U45.4
- net N$192: now also U46.6, U47.1; no longer U46.5, U47.3
- net N$193: now also U46.5, U47.2; no longer U46.6, U47.4
- net N$194: now also U47.6, U48.1; no longer U47.5, U48.3
- net N$195: now also U47.5, U48.2; no longer U47.6, U48.4
- net N$196: now also U48.6, U49.1; no longer U48.5, U49.3
- net N$197: now also U48.5, U49.2; no longer U48.6, U49.4
- net N$198: now also U49.6, U50.1; no longer U49.5, U50.3
- net N$199: now also U49.5, U50.2; no longer U49.6, U50.4
- net N$202: now also U50.6, U51.1; no longer U50.5, U51.3
- net N$203: now also U50.5, U51.2; no longer U50.6, U51.4
- net N$204: now also U51.6, U52.1; no longer U51.5, U52.3
- net N$205: now also U51.5, U52.2; no longer U51.6, U52.4
- net N$206: now also U52.6, U53.1; no longer U52.5, U53.3
- net N$207: now also U52.5, U53.2; no longer U52.6, U53.4
- net N$208: now also U54.6, U55.1; no longer U54.5, U55.3
- net N$209: now also U54.5, U55.2; no longer U54.6, U55.4
- net N$210: now also U55.6, U56.1; no longer U55.5, U56.3
- net N$211: now also U55.5, U56.2; no longer U55.6, U56.4
- net N$212: now also U56.6, U57.1; no longer U56.5, U57.3
- net N$213: now also U56.5, U57.2; no longer U56.6, U57.4
- net N$214: now also U57.6, U58.1; no longer U57.5, U58.3
- net N$215: now also U57.5, U58.2; no longer U57.6, U58.4
- net N$216: now also U58.6, U59.1; no longer U58.5, U59.3
- net N$217: now also U58.5, U59.2; no longer U58.6, U59.4
- net N$218: now also U59.6, U60.1; no longer U59.5, U60.3
- net N$219: now also U59.5, U60.2; no longer U59.6, U60.4
- net N$220: now also U6.6, U7.1; no longer U6.5, U7.3
- net N$221: now also U6.5, U7.2; no longer U6.6, U7.4
- net N$222: now also U60.6, U61.1; no longer U60.5, U61.3
- net N$223: now also U60.5, U61.2; no longer U60.6, U61.4
- net N$224: now also U62.6, U63.1; no longer U62.5, U63.3
- net N$225: now also U62.5, U63.2; no longer U62.6, U63.4
- net N$226: now also U63.6, U64.1; no longer U63.5, U64.3
- net N$227: now also U63.5, U64.2; no longer U63.6, U64.4
- net N$228: now also U64.6, U65.1; no longer U64.5, U65.3
- net N$229: now also U64.5, U65.2; no longer U64.6, U65.4
- net N$230: now also U65.6, U66.1; no longer U65.5, U66.3
- net N$231: now also U65.5, U66.2; no longer U65.6, U66.4
- net N$232: now also U66.6, U67.1; no longer U66.5, U67.3
- net N$233: now also U66.5, U67.2; no longer U66.6, U67.4
- net N$234: now also U67.6, U68.1; no longer U67.5, U68.3
- net N$235: now also U67.5, U68.2; no longer U67.6, U68.4
- net N$236: now also U68.6, U69.1; no longer U68.5, U69.3
- net N$237: now also U68.5, U69.2; no longer U68.6, U69.4
- net N$238: now also U7.6, U8.1; no longer U7.5, U8.3
- net N$239: now also U7.5, U8.2; no longer U7.6, U8.4
- net N$240: now also U8.6, U9.1; no longer U8.5, U9.3
- net N$241: now also U8.5, U9.2; no longer U8.6, U9.4

Commit message: Refactor chessboard hardware around modular KiCad design
Parts:
- removed RS1: KSK-1A66-1015, symbol Generated:RS1
- removed RS10: KSK-1A66-1015, symbol Generated:RS10
- removed RS11: KSK-1A66-1015, symbol Generated:RS11
- removed RS12: KSK-1A66-1015, symbol Generated:RS12
- removed RS13: KSK-1A66-1015, symbol Generated:RS13
- removed RS14: KSK-1A66-1015, symbol Generated:RS14
- removed RS15: KSK-1A66-1015, symbol Generated:RS15
- removed RS16: KSK-1A66-1015, symbol Generated:RS16
- removed RS17: KSK-1A66-1015, symbol Generated:RS17
- removed RS18: KSK-1A66-1015, symbol Generated:RS18
- removed RS19: KSK-1A66-1015, symbol Generated:RS19
- removed RS2: KSK-1A66-1015, symbol Generated:RS2
- removed RS20: KSK-1A66-1015, symbol Generated:RS20
- removed RS21: KSK-1A66-1015, symbol Generated:RS21
- removed RS22: KSK-1A66-1015, symbol Generated:RS22
- removed RS23: KSK-1A66-1015, symbol Generated:RS23
- removed RS24: KSK-1A66-1015, symbol Generated:RS24
- removed RS25: KSK-1A66-1015, symbol Generated:RS25
- removed RS26: KSK-1A66-1015, symbol Generated:RS26
- removed RS27: KSK-1A66-1015, symbol Generated:RS27
- removed RS28: KSK-1A66-1015, symbol Generated:RS28
- removed RS29: KSK-1A66-1015, symbol Generated:RS29
- removed RS3: KSK-1A66-1015, symbol Generated:RS3
- removed RS30: KSK-1A66-1015, symbol Generated:RS30
- removed RS31: KSK-1A66-1015, symbol Generated:RS31
- removed RS32: KSK-1A66-1015, symbol Generated:RS32
- removed RS33: KSK-1A66-1015, symbol Generated:RS33
- removed RS34: KSK-1A66-1015, symbol Generated:RS34
- removed RS35: KSK-1A66-1015, symbol Generated:RS35
- removed RS36: KSK-1A66-1015, symbol Generated:RS36
- removed RS37: KSK-1A66-1015, symbol Generated:RS37
- removed RS38: KSK-1A66-1015, symbol Generated:RS38
- removed RS39: KSK-1A66-1015, symbol Generated:RS39
- removed RS4: KSK-1A66-1015, symbol Generated:RS4
- removed RS40: KSK-1A66-1015, symbol Generated:RS40
- removed RS41: KSK-1A66-1015, symbol Generated:RS41
- removed RS42: KSK-1A66-1015, symbol Generated:RS42
- removed RS43: KSK-1A66-1015, symbol Generated:RS43
- removed RS44: KSK-1A66-1015, symbol Generated:RS44
- removed RS45: KSK-1A66-1015, symbol Generated:RS45
- removed RS46: KSK-1A66-1015, symbol Generated:RS46
- removed RS47: KSK-1A66-1015, symbol Generated:RS47
- removed RS48: KSK-1A66-1015, symbol Generated:RS48
- removed RS49: KSK-1A66-1015, symbol Generated:RS49
- removed RS5: KSK-1A66-1015, symbol Generated:RS5
- removed RS50: KSK-1A66-1015, symbol Generated:RS50
- removed RS51: KSK-1A66-1015, symbol Generated:RS51
- removed RS52: KSK-1A66-1015, symbol Generated:RS52
- removed RS53: KSK-1A66-1015, symbol Generated:RS53
- removed RS54: KSK-1A66-1015, symbol Generated:RS54
- removed RS55: KSK-1A66-1015, symbol Generated:RS55
- removed RS56: KSK-1A66-1015, symbol Generated:RS56
- removed RS57: KSK-1A66-1015, symbol Generated:RS57
- removed RS58: KSK-1A66-1015, symbol Generated:RS58
- removed RS59: KSK-1A66-1015, symbol Generated:RS59
- removed RS6: KSK-1A66-1015, symbol Generated:RS6
- removed RS60: KSK-1A66-1015, symbol Generated:RS60
- removed RS61: KSK-1A66-1015, symbol Generated:RS61
- removed RS62: KSK-1A66-1015, symbol Generated:RS62
- removed RS63: KSK-1A66-1015, symbol Generated:RS63
- removed RS64: KSK-1A66-1015, symbol Generated:RS64
- removed RS7: KSK-1A66-1015, symbol Generated:RS7
- removed RS8: KSK-1A66-1015, symbol Generated:RS8
- removed RS9: KSK-1A66-1015, symbol Generated:RS9
- added C100: CC0603KRX7R9BB104, symbol Generated:C100
- added C101: CC0603KRX7R9BB104, symbol Generated:C101
- added C102: CC0603KRX7R9BB104, symbol Generated:C102
- added C103: CC0603KRX7R9BB104, symbol Generated:C103
- added C104: CC0603KRX7R9BB104, symbol Generated:C104
- added C105: CC0603KRX7R9BB104, symbol Generated:C105
- added C106: CC0603KRX7R9BB104, symbol Generated:C106
- added C107: CC0603KRX7R9BB104, symbol Generated:C107
- added C108: CC0603KRX7R9BB104, symbol Generated:C108
- added C109: CC0603KRX7R9BB104, symbol Generated:C109
- added C110: CC0603KRX7R9BB104, symbol Generated:C110
- added C111: CC0603KRX7R9BB104, symbol Generated:C111
- added C112: CC0603KRX7R9BB104, symbol Generated:C112
- added C113: CC0603KRX7R9BB104, symbol Generated:C113
- added C114: CC0603KRX7R9BB104, symbol Generated:C114
- added C115: CC0603KRX7R9BB104, symbol Generated:C115
- added C116: CC0603KRX7R9BB104, symbol Generated:C116
- added C117: CC0603KRX7R9BB104, symbol Generated:C117
- added C118: CC0603KRX7R9BB104, symbol Generated:C118
- added C119: CC0603KRX7R9BB104, symbol Generated:C119
- added C120: CC0603KRX7R9BB104, symbol Generated:C120
- added C121: CC0603KRX7R9BB104, symbol Generated:C121
- added C122: CC0603KRX7R9BB104, symbol Generated:C122
- added C123: CC0603KRX7R9BB104, symbol Generated:C123
- added C124: CC0603KRX7R9BB104, symbol Generated:C124
- added C125: CC0603KRX7R9BB104, symbol Generated:C125
- added C126: CC0603KRX7R9BB104, symbol Generated:C126
- added C127: CC0603KRX7R9BB104, symbol Generated:C127
- added C128: CC0603KRX7R9BB104, symbol Generated:C128
- added C129: CC0603KRX7R9BB104, symbol Generated:C129
- added C130: CC0603KRX7R9BB104, symbol Generated:C130
- added C131: CC0603KRX7R9BB104, symbol Generated:C131
- added C132: CC0603KRX7R9BB104, symbol Generated:C132
- added C133: CC0603KRX7R9BB104, symbol Generated:C133
- added C134: CC0603KRX7R9BB104, symbol Generated:C134
- added C135: CC0603KRX7R9BB104, symbol Generated:C135
- added C72: CC0603KRX7R9BB104, symbol Generated:C72
- added C73: CC0603KRX7R9BB104, symbol Generated:C73
- added C74: CC0603KRX7R9BB104, symbol Generated:C74
- added C75: CC0603KRX7R9BB104, symbol Generated:C75
- added C76: CC0603KRX7R9BB104, symbol Generated:C76
- added C77: CC0603KRX7R9BB104, symbol Generated:C77
- added C78: CC0603KRX7R9BB104, symbol Generated:C78
- added C79: CC0603KRX7R9BB104, symbol Generated:C79
- added C80: CC0603KRX7R9BB104, symbol Generated:C80
- added C81: CC0603KRX7R9BB104, symbol Generated:C81
- added C82: CC0603KRX7R9BB104, symbol Generated:C82
- added C83: CC0603KRX7R9BB104, symbol Generated:C83
- added C84: CC0603KRX7R9BB104, symbol Generated:C84
- added C85: CC0603KRX7R9BB104, symbol Generated:C85
- added C86: CC0603KRX7R9BB104, symbol Generated:C86
- added C87: CC0603KRX7R9BB104, symbol Generated:C87
- added C88: CC0603KRX7R9BB104, symbol Generated:C88
- added C89: CC0603KRX7R9BB104, symbol Generated:C89
- added C90: CC0603KRX7R9BB104, symbol Generated:C90
- added C91: CC0603KRX7R9BB104, symbol Generated:C91
- added C92: CC0603KRX7R9BB104, symbol Generated:C92
- added C93: CC0603KRX7R9BB104, symbol Generated:C93
- added C94: CC0603KRX7R9BB104, symbol Generated:C94
- added C95: CC0603KRX7R9BB104, symbol Generated:C95
- added C96: CC0603KRX7R9BB104, symbol Generated:C96
- added C97: CC0603KRX7R9BB104, symbol Generated:C97
- added C98: CC0603KRX7R9BB104, symbol Generated:C98
- added C99: CC0603KRX7R9BB104, symbol Generated:C99
- added HS1: DRV5032FCDBZR, symbol Generated:HS1
- added HS10: DRV5032FCDBZR, symbol Generated:HS10
- added HS11: DRV5032FCDBZR, symbol Generated:HS11
- added HS12: DRV5032FCDBZR, symbol Generated:HS12
- added HS13: DRV5032FCDBZR, symbol Generated:HS13
- added HS14: DRV5032FCDBZR, symbol Generated:HS14
- added HS15: DRV5032FCDBZR, symbol Generated:HS15
- added HS16: DRV5032FCDBZR, symbol Generated:HS16
- added HS17: DRV5032FCDBZR, symbol Generated:HS17
- added HS18: DRV5032FCDBZR, symbol Generated:HS18
- added HS19: DRV5032FCDBZR, symbol Generated:HS19
- added HS2: DRV5032FCDBZR, symbol Generated:HS2
- added HS20: DRV5032FCDBZR, symbol Generated:HS20
- added HS21: DRV5032FCDBZR, symbol Generated:HS21
- added HS22: DRV5032FCDBZR, symbol Generated:HS22
- added HS23: DRV5032FCDBZR, symbol Generated:HS23
- added HS24: DRV5032FCDBZR, symbol Generated:HS24
- added HS25: DRV5032FCDBZR, symbol Generated:HS25
- added HS26: DRV5032FCDBZR, symbol Generated:HS26
- added HS27: DRV5032FCDBZR, symbol Generated:HS27
- added HS28: DRV5032FCDBZR, symbol Generated:HS28
- added HS29: DRV5032FCDBZR, symbol Generated:HS29
- added HS3: DRV5032FCDBZR, symbol Generated:HS3
- added HS30: DRV5032FCDBZR, symbol Generated:HS30
- added HS31: DRV5032FCDBZR, symbol Generated:HS31
- added HS32: DRV5032FCDBZR, symbol Generated:HS32
- added HS33: DRV5032FCDBZR, symbol Generated:HS33
- added HS34: DRV5032FCDBZR, symbol Generated:HS34
- added HS35: DRV5032FCDBZR, symbol Generated:HS35
- added HS36: DRV5032FCDBZR, symbol Generated:HS36
- added HS37: DRV5032FCDBZR, symbol Generated:HS37
- added HS38: DRV5032FCDBZR, symbol Generated:HS38
- added HS39: DRV5032FCDBZR, symbol Generated:HS39
- added HS4: DRV5032FCDBZR, symbol Generated:HS4
- added HS40: DRV5032FCDBZR, symbol Generated:HS40
- added HS41: DRV5032FCDBZR, symbol Generated:HS41
- added HS42: DRV5032FCDBZR, symbol Generated:HS42
- added HS43: DRV5032FCDBZR, symbol Generated:HS43
- added HS44: DRV5032FCDBZR, symbol Generated:HS44
- added HS45: DRV5032FCDBZR, symbol Generated:HS45
- added HS46: DRV5032FCDBZR, symbol Generated:HS46
- added HS47: DRV5032FCDBZR, symbol Generated:HS47
- added HS48: DRV5032FCDBZR, symbol Generated:HS48
- added HS49: DRV5032FCDBZR, symbol Generated:HS49
- added HS5: DRV5032FCDBZR, symbol Generated:HS5
- added HS50: DRV5032FCDBZR, symbol Generated:HS50
- added HS51: DRV5032FCDBZR, symbol Generated:HS51
- added HS52: DRV5032FCDBZR, symbol Generated:HS52
- added HS53: DRV5032FCDBZR, symbol Generated:HS53
- added HS54: DRV5032FCDBZR, symbol Generated:HS54
- added HS55: DRV5032FCDBZR, symbol Generated:HS55
- added HS56: DRV5032FCDBZR, symbol Generated:HS56
- added HS57: DRV5032FCDBZR, symbol Generated:HS57
- added HS58: DRV5032FCDBZR, symbol Generated:HS58
- added HS59: DRV5032FCDBZR, symbol Generated:HS59
- added HS6: DRV5032FCDBZR, symbol Generated:HS6
- added HS60: DRV5032FCDBZR, symbol Generated:HS60
- added HS61: DRV5032FCDBZR, symbol Generated:HS61
- added HS62: DRV5032FCDBZR, symbol Generated:HS62
- added HS63: DRV5032FCDBZR, symbol Generated:HS63
- added HS64: DRV5032FCDBZR, symbol Generated:HS64
- added HS7: DRV5032FCDBZR, symbol Generated:HS7
- added HS8: DRV5032FCDBZR, symbol Generated:HS8
- added HS9: DRV5032FCDBZR, symbol Generated:HS9
- C1: value EEU-FR1A102 -> 10ZLJ1000M10X16
- C10, C11, C12, C13, C14, C15, C16, C17, C18, C19, C20, C21, C22, C23, C24, C25, C26, C27, C28, C29, C3, C30, C31, C32, C33, C34, C35, C36, C37, C38, C39, C4, C40, C41, C42, C43, C44, C45, C46, C47, C48, C49, C5, C50, C51, C52, C53, C54, C55, C56, C57, C58, C59, C6, C60, C61, C62, C63, C64, C65, C66, C67, C68, C69, C7, C70, C71, C8, C9: value C315C104M5U5TA -> CC0603KRX7R9BB104
- C2: value UVR1C100MDD -> CC0805KKX5R6BB106
- D1: value P6KE6.8A -> SMBJ6.0A
- F1: value 3557 -> 0453005.MR
- J1: value SSW-120-02-G-D -> PPPC202LFBN-RC
- J2: value SSW-104-02-G-S -> PPPC041LFBN-RC
- R1, R2: value MFR-25FBF52-4K7 -> RC0603FR-074K7L
- SW1, SW10, SW11, SW12, SW2, SW3, SW4, SW5, SW6, SW7, SW8, SW9: value B3F-4050 -> TL1105SPF100QG
- TP1, TP2, TP3, TP4: value 1502-2 -> S1751-46R
- U1, U2, U3, U4: value MCP23017-E/SP -> MCP23017-E/SO
- U5: value SN74AHCT125N -> SN74AHCT125DR
Connections:
- net +3V3: now also C100.1, C101.1, C102.1, C103.1, C104.1, C105.1, C106.1, C107.1, C108.1, C109.1, C110.1, C111.1, C112.1, C113.1, C114.1, C115.1, C116.1, C117.1, C118.1, C119.1, C120.1, C121.1, C122.1, C123.1, C124.1, C125.1, C126.1, C127.1, C128.1, C129.1, C130.1, C131.1, C132.1, C133.1, C134.1, C135.1, C72.1, C73.1, C74.1, C75.1, C76.1, C77.1, C78.1, C79.1, C80.1, C81.1, C82.1, C83.1, C84.1, C85.1, C86.1, C87.1, C88.1, C89.1, C90.1, C91.1, C92.1, C93.1, C94.1, C95.1, C96.1, C97.1, C98.1, C99.1, HS1.1, HS10.1, HS11.1, HS12.1, HS13.1, HS14.1, HS15.1, HS16.1, HS17.1, HS18.1, HS19.1, HS2.1, HS20.1, HS21.1, HS22.1, HS23.1, HS24.1, HS25.1, HS26.1, HS27.1, HS28.1, HS29.1, HS3.1, HS30.1, HS31.1, HS32.1, HS33.1, HS34.1, HS35.1, HS36.1, HS37.1, HS38.1, HS39.1, HS4.1, HS40.1, HS41.1, HS42.1, HS43.1, HS44.1, HS45.1, HS46.1, HS47.1, HS48.1, HS49.1, HS5.1, HS50.1, HS51.1, HS52.1, HS53.1, HS54.1, HS55.1, HS56.1, HS57.1, HS58.1, HS59.1, HS6.1, HS60.1, HS61.1, HS62.1, HS63.1, HS64.1, HS7.1, HS8.1, HS9.1
- net GND: now also C100.2, C101.2, C102.2, C103.2, C104.2, C105.2, C106.2, C107.2, C108.2, C109.2, C110.2, C111.2, C112.2, C113.2, C114.2, C115.2, C116.2, C117.2, C118.2, C119.2, C120.2, C121.2, C122.2, C123.2, C124.2, C125.2, C126.2, C127.2, C128.2, C129.2, C130.2, C131.2, C132.2, C133.2, C134.2, C135.2, C72.2, C73.2, C74.2, C75.2, C76.2, C77.2, C78.2, C79.2, C80.2, C81.2, C82.2, C83.2, C84.2, C85.2, C86.2, C87.2, C88.2, C89.2, C90.2, C91.2, C92.2, C93.2, C94.2, C95.2, C96.2, C97.2, C98.2, C99.2, HS1.3, HS10.3, HS11.3, HS12.3, HS13.3, HS14.3, HS15.3, HS16.3, HS17.3, HS18.3, HS19.3, HS2.3, HS20.3, HS21.3, HS22.3, HS23.3, HS24.3, HS25.3, HS26.3, HS27.3, HS28.3, HS29.3, HS3.3, HS30.3, HS31.3, HS32.3, HS33.3, HS34.3, HS35.3, HS36.3, HS37.3, HS38.3, HS39.3, HS4.3, HS40.3, HS41.3, HS42.3, HS43.3, HS44.3, HS45.3, HS46.3, HS47.3, HS48.3, HS49.3, HS5.3, HS50.3, HS51.3, HS52.3, HS53.3, HS54.3, HS55.3, HS56.3, HS57.3, HS58.3, HS59.3, HS6.3, HS60.3, HS61.3, HS62.3, HS63.3, HS64.3, HS7.3, HS8.3, HS9.3
- net SQ_A1: now also HS1.2
- net SQ_A2: now also HS5.2
- net SQ_A3: now also HS9.2
- net SQ_A4: now also HS13.2
- net SQ_A5: now also HS33.2
- net SQ_A6: now also HS37.2
- net SQ_A7: now also HS41.2
- net SQ_A8: now also HS45.2
- net SQ_B1: now also HS2.2
- net SQ_B2: now also HS6.2
- net SQ_B3: now also HS10.2
- net SQ_B4: now also HS14.2
- net SQ_B5: now also HS34.2
- net SQ_B6: now also HS38.2
- net SQ_B7: now also HS42.2
- net SQ_B8: now also HS46.2
- net SQ_C1: now also HS3.2
- net SQ_C2: now also HS7.2
- net SQ_C3: now also HS11.2
- net SQ_C4: now also HS15.2
- net SQ_C5: now also HS35.2
- net SQ_C6: now also HS39.2
- net SQ_C7: now also HS43.2
- net SQ_C8: now also HS47.2
- net SQ_D1: now also HS4.2
- net SQ_D2: now also HS8.2
- net SQ_D3: now also HS12.2
- net SQ_D4: now also HS16.2
- net SQ_D5: now also HS36.2
- net SQ_D6: now also HS40.2
- net SQ_D7: now also HS44.2
- net SQ_D8: now also HS48.2
- net SQ_E1: now also HS17.2
- net SQ_E2: now also HS21.2
- net SQ_E3: now also HS25.2
- net SQ_E4: now also HS29.2
- net SQ_E5: now also HS49.2
- net SQ_E6: now also HS53.2
- net SQ_E7: now also HS57.2
- net SQ_E8: now also HS61.2
- net SQ_F1: now also HS18.2
- net SQ_F2: now also HS22.2
- net SQ_F3: now also HS26.2
- net SQ_F4: now also HS30.2
- net SQ_F5: now also HS50.2
- net SQ_F6: now also HS54.2
- net SQ_F7: now also HS58.2
- net SQ_F8: now also HS62.2
- net SQ_G1: now also HS19.2
- net SQ_G2: now also HS23.2
- net SQ_G3: now also HS27.2
- net SQ_G4: now also HS31.2
- net SQ_G5: now also HS51.2
- net SQ_G6: now also HS55.2
- net SQ_G7: now also HS59.2
- net SQ_G8: now also HS63.2
- net SQ_H1: now also HS20.2
- net SQ_H2: now also HS24.2
- net SQ_H3: now also HS28.2
- net SQ_H4: now also HS32.2
- net SQ_H5: now also HS52.2
- net SQ_H6: now also HS56.2
- net SQ_H7: now also HS60.2
- net SQ_H8: now also HS64.2
Other:
- moved on the sheet: C10, C11, C12, C13, C14, C15, C16, C17, C18, C19, C2, C20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
