File: hardware/pcb/generated/chess-board.kicad_sch (KiCad schematic)
At the start: 292 parts, among them J1 PPPC202LFBN-RC, J2 PPPC041LFBN-RC, J3 PJ-102A, SW1 TL1105SPF100QG, SW10 TL1105SPF100QG, SW11 TL1105SPF100QG, SW12 TL1105SPF100QG, SW13 RA11131100, SW2 TL1105SPF100QG, SW3 TL1105SPF100QG, SW4 TL1105SPF100QG, SW5 TL1105SPF100QG, SW6 TL1105SPF100QG, SW7 TL1105SPF100QG, SW8 TL1105SPF100QG, SW9 TL1105SPF100QG, U1 MCP23017-E/SO, U10 SK9822-EC20, U11 SK9822-EC20, U12 SK9822-EC20, U13 SK9822-EC20, U14 SK9822-EC20, U15 SK9822-EC20, U16 SK9822-EC20, U17 SK9822-EC20, U18 SK9822-EC20, U19 SK9822-EC20, U2 MCP23017-E/SO, U20 SK9822-EC20, U21 SK9822-EC20, U22 SK9822-EC20, U23 SK9822-EC20, U24 SK9822-EC20, U25 SK9822-EC20, U26 SK9822-EC20, U27 SK9822-EC20, U28 SK9822-EC20, U29 SK9822-EC20, U3 MCP23017-E/SO, U30 SK9822-EC20, U31 SK9822-EC20, U32 SK9822-EC20, U33 SK9822-EC20, U34 SK9822-EC20, U35 SK9822-EC20, U36 SK9822-EC20, U37 SK9822-EC20, U38 SK9822-EC20, U39 SK9822-EC20, U4 MCP23017-E/SO, U40 SK9822-EC20, U41 SK9822-EC20, U42 SK9822-EC20, U43 SK9822-EC20, U44 SK9822-EC20, U45 SK9822-EC20, U46 SK9822-EC20, U47 SK9822-EC20, U48 SK9822-EC20, U49 SK9822-EC20, U5 SN74AHCT125DR, U50 SK9822-EC20, U51 SK9822-EC20, U52 SK9822-EC20, U53 SK9822-EC20, U54 SK9822-EC20, U55 SK9822-EC20, U56 SK9822-EC20, U57 SK9822-EC20, U58 SK9822-EC20, U59 SK9822-EC20, U6 SK9822-EC20, U60 SK9822-EC20, U61 SK9822-EC20, U62 SK9822-EC20, U63 SK9822-EC20, U64 SK9822-EC20, U65 SK9822-EC20, U66 SK9822-EC20, U67 SK9822-EC20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

Commit message: fix(pcb): harden fabrication release design
Parts:
- added R3: RC0603FR-074K7L, symbol Generated:R3
- added TP5: S1751-46R, symbol Generated:TP5
- added TP6: S1751-46R, symbol Generated:TP6
- added TP7: S1751-46R, symbol Generated:TP7
- added TP8: S1751-46R, symbol Generated:TP8
- F1: value 0453005.MR -> 0453002.MR
Connections:
- net +3V3: now also R3.1, TP5.1
- net I2C_SCL: now also TP6.1
- net I2C_SDA: now also TP7.1
- net SENSE_IRQ: now also R3.2, TP8.1
Other:
- moved on the sheet: SW1, SW10, SW11, SW12, SW13, SW2, SW3, SW4, SW5, SW6, SW7, SW8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
