File: hardware/pcb/generated/chess-board.kicad_sch (KiCad schematic)
At the start: 297 parts, among them J1 PPPC202LFBN-RC, J2 PPPC041LFBN-RC, J3 PJ-102A, SW1 TL1105SPF100QG, SW10 TL1105SPF100QG, SW11 TL1105SPF100QG, SW12 TL1105SPF100QG, SW13 RA11131100, SW2 TL1105SPF100QG, SW3 TL1105SPF100QG, SW4 TL1105SPF100QG, SW5 TL1105SPF100QG, SW6 TL1105SPF100QG, SW7 TL1105SPF100QG, SW8 TL1105SPF100QG, SW9 TL1105SPF100QG, U1 MCP23017-E/SO, U10 SK9822-EC20, U11 SK9822-EC20, U12 SK9822-EC20, U13 SK9822-EC20, U14 SK9822-EC20, U15 SK9822-EC20, U16 SK9822-EC20, U17 SK9822-EC20, U18 SK9822-EC20, U19 SK9822-EC20, U2 MCP23017-E/SO, U20 SK9822-EC20, U21 SK9822-EC20, U22 SK9822-EC20, U23 SK9822-EC20, U24 SK9822-EC20, U25 SK9822-EC20, U26 SK9822-EC20, U27 SK9822-EC20, U28 SK9822-EC20, U29 SK9822-EC20, U3 MCP23017-E/SO, U30 SK9822-EC20, U31 SK9822-EC20, U32 SK9822-EC20, U33 SK9822-EC20, U34 SK9822-EC20, U35 SK9822-EC20, U36 SK9822-EC20, U37 SK9822-EC20, U38 SK9822-EC20, U39 SK9822-EC20, U4 MCP23017-E/SO, U40 SK9822-EC20, U41 SK9822-EC20, U42 SK9822-EC20, U43 SK9822-EC20, U44 SK9822-EC20, U45 SK9822-EC20, U46 SK9822-EC20, U47 SK9822-EC20, U48 SK9822-EC20, U49 SK9822-EC20, U5 SN74AHCT125DR, U50 SK9822-EC20, U51 SK9822-EC20, U52 SK9822-EC20, U53 SK9822-EC20, U54 SK9822-EC20, U55 SK9822-EC20, U56 SK9822-EC20, U57 SK9822-EC20, U58 SK9822-EC20, U59 SK9822-EC20, U6 SK9822-EC20, U60 SK9822-EC20, U61 SK9822-EC20, U62 SK9822-EC20, U63 SK9822-EC20, U64 SK9822-EC20, U65 SK9822-EC20, U66 SK9822-EC20, U67 SK9822-EC20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

Commit message: Standardize PCB generation rules
Other:
- title: Code-composed chess board -> Chess Smart Board - Single Board Electronics
Changed lines of the file:
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@@
   (paper "A0")
   (title_block
-    (title "Code-composed chess board")
-    (rev "B-PROTOTYPE")
+    (title "Chess Smart Board - Single Board Electronics")
+    (rev "C-PROTOTYPE")
     (company "Chess")
     (comment 1 "Generated from board/netlist.json; do not hand edit")

Commit message: chore(hardware): refresh PCB and firmware outputs
Parts:
- removed R3: RC0603FR-074K7L, symbol Generated:R3
- removed TP8: S1751-46R, symbol Generated:TP8
- added C136: CC0603KRX7R9BB104, symbol Generated:C136
- added C137: CC0603KRX7R9BB104, symbol Generated:C137
- added C138: CC0603KRX7R9BB104, symbol Generated:C138
- added C139: CC0603KRX7R9BB104, symbol Generated:C139
- added U70: TCA9554DWR, symbol Generated:U70
- added U71: TCA9554DWR, symbol Generated:U71
- added U72: TCA9554DWR, symbol Generated:U72
- added U73: TCA9554DWR, symbol Generated:U73
- U1, U2, U3, U4: value MCP23017-E/SO -> TCA9554DWR
Connections:
- net N$187 is gone; now on net N$174: U42.5, U43.2
- net N$188 is gone; now on net N$175: U43.6, U44.1
- net N$229 is gone; now on net N$216: U64.5, U65.2
- net N$230 is gone; now on net N$217: U65.6, U66.1
- net N$231 is gone; now on net N$218: U65.5, U66.2
- net N$232 is gone; now on net N$219: U66.6, U67.1
- net N$233 is gone; now on net N$220: U66.5, U67.2
- net N$234 is gone; now on net N$221: U67.6, U68.1
- net N$235 is gone; now on net N$222: U67.5, U68.2
- net N$236 is gone; now on net N$223: U68.6, U69.1
- net N$237 is gone; now on net N$224: U68.5, U69.2
- net N$238 is gone; now on net N$225: U7.6, U8.1
- net N$239 is gone; now on net N$226: U7.5, U8.2
- net N$240 is gone; now on net N$227: U8.6, U9.1
- net N$241 is gone; now on net N$228: U8.5, U9.2
- net +3V3: now also U1.16, U2.1, U2.16, U3.2, U4.1, U4.2, C136.1, C137.1, C138.1, C139.1, U70.16, U70.3, U71.1, U71.16, U71.3, U72.16, U72.2, U72.3, U73.1, U73.16, U73.2, U73.3; no longer U1.18, U1.9, U2.15, U2.18, U2.9, U3.18, U3.9, U4.15, U4.18, U4.9
- net GND: now also U1.1, U1.2, U1.3, U1.8, U2.2, U2.3, U2.8, U3.1, U3.3, U3.8, U4.3, U4.8, C136.2, C137.2, C138.2, C139.2, U70.1, U70.2, U70.8, U71.2, U71.8, U72.1, U72.8, U73.8; no longer U1.10, U1.15, U1.16, U1.17, U2.10, U2.16, U2.17, U3.10, U3.15, U3.17, U4.10, U4.17
- net I2C_SCL: now also U1.14, U2.14, U3.14, U4.14, U70.14, U71.14, U72.14, U73.14; no longer U1.12, U2.12, U3.12, U4.12
- net I2C_SDA: now also U1.15, U2.15, U3.15, U4.15, U70.15, U71.15, U72.15, U73.15; no longer U1.13, U2.13, U3.13, U4.13
- net N$119: now also U11.6, U12.1; no longer U10.1, U9.6
- net N$120: now also U11.5, U12.2; no longer U10.2, U9.5
- net N$121: now also U12.6, U13.1; no longer U10.6, U11.1
- net N$122: now also U12.5, U13.2; no longer U10.5, U11.2
- net N$123: now also U14.6, U15.1; no longer U11.6, U12.1
- net N$124: now also U14.5, U15.2; no longer U11.5, U12.2
- net N$125: now also U15.6, U16.1; no longer U12.6, U13.1
- net N$126: now also U15.5, U16.2; no longer U12.5, U13.2
- net N$127: now also U16.6, U17.1; no longer U14.6, U15.1
- net N$128: now also U16.5, U17.2; no longer U14.5, U15.2
- net N$129: now also U17.6, U18.1; no longer U15.6, U16.1
- net N$130: now also U17.5, U18.2; no longer U15.5, U16.2
- net N$131: now also U18.6, U19.1; no longer U16.6, U17.1
- net N$132: now also U18.5, U19.2; no longer U16.5, U17.2
- net N$133: now also U19.6, U20.1; no longer U17.6, U18.1
- net N$134: now also U19.5, U20.2; no longer U17.5, U18.2
- net N$135: now also U20.6, U21.1; no longer U18.6, U19.1
- net N$136: now also U20.5, U21.2; no longer U18.5, U19.2
- net N$137: now also U22.6, U23.1; no longer U19.6, U20.1
- net N$138: now also U22.5, U23.2; no longer U19.5, U20.2
- net N$142: now also U24.5, U25.2; no longer U20.6, U21.1
- net N$143: now also U25.6, U26.1; no longer U20.5, U21.2
- net N$144: now also U25.5, U26.2; no longer U22.6, U23.1
- net N$145: now also U26.6, U27.1; no longer U22.5, U23.2
- net N$146: now also U26.5, U27.2; no longer U23.6, U24.1
- net N$147: now also U27.6, U28.1; no longer U23.5, U24.2
- net N$148: now also U27.5, U28.2; no longer U24.6, U25.1
- net N$149: now also U28.6, U29.1; no longer U24.5, U25.2
- net N$150: now also U28.5, U29.2; no longer U25.6, U26.1
- net N$151: now also U30.6, U31.1; no longer U25.5, U26.2
- net N$152: now also U30.5, U31.2; no longer U26.6, U27.1
- net N$153: now also U31.6, U32.1; no longer U26.5, U27.2
- net N$154: now also U31.5, U32.2; no longer U27.6, U28.1
- net N$155: now also U32.6, U33.1; no longer U27.5, U28.2
- net N$156: now also U32.5, U33.2; no longer U28.6, U29.1
- net N$157: now also U33.6, U34.1; no longer U28.5, U29.2
- net N$161: now also U35.6, U36.1; no longer U30.6, U31.1
- net N$162: now also U35.5, U36.2; no longer U30.5, U31.2
- net N$163: now also U36.6, U37.1; no longer U31.6, U32.1
- net N$164: now also U36.5, U37.2; no longer U31.5, U32.2
- net N$165: now also U38.6, U39.1; no longer U32.6, U33.1
- net N$166: now also U38.5, U39.2; no longer U32.5, U33.2
- net N$167: now also U39.6, U40.1; no longer U33.6, U34.1
- net N$168: now also U39.5, U40.2; no longer U33.5, U34.2
- net N$169: now also U40.6, U41.1; no longer U34.6, U35.1
- net N$170: now also U40.5, U41.2; no longer U34.5, U35.2
- net N$171: now also U41.6, U42.1; no longer U35.6, U36.1
- net N$172: now also U41.5, U42.2; no longer U35.5, U36.2
- net N$173: now also U42.6, U43.1; no longer U36.6, U37.1
- net N$174: no longer U36.5, U37.2
- net N$175: no longer U38.6, U39.1
- net N$176: now also U43.5, U44.2; no longer U38.5, U39.2
- net N$177: now also U44.6, U45.1; no longer U39.6, U40.1
- net N$178: now also U44.5, U45.2; no longer U39.5, U40.2
- net N$182: now also U47.5, U48.2; no longer U40.6, U41.1
- net N$183: now also U48.6, U49.1; no longer U40.5, U41.2
- net N$184: now also U48.5, U49.2; no longer U41.6, U42.1
- net N$185: now also U49.6, U50.1; no longer U41.5, U42.2
- net N$186: now also U49.5, U50.2; no longer U42.6, U43.1
- net N$189: now also U50.6, U51.1; no longer U43.5, U44.2
- net N$190: now also U50.5, U51.2; no longer U44.6, U45.1
- net N$191: now also U51.6, U52.1; no longer U44.5, U45.2
- net N$192: now also U51.5, U52.2; no longer U46.6, U47.1
- net N$193: now also U52.6, U53.1; no longer U46.5, U47.2
- net N$194: now also U52.5, U53.2; no longer U47.6, U48.1
- net N$195: now also U54.6, U55.1; no longer U47.5, U48.2
- net N$196: now also U54.5, U55.2; no longer U48.6, U49.1
- net N$197: now also U55.6, U56.1; no longer U48.5, U49.2
- net N$198: now also U55.5, U56.2; no longer U49.6, U50.1
- net N$199: now also U56.6, U57.1; no longer U49.5, U50.2
- net N$202: now also U57.5, U58.2; no longer U50.6, U51.1
- net N$203: now also U58.6, U59.1; no longer U50.5, U51.2
- net N$204: now also U58.5, U59.2; no longer U51.6, U52.1
- net N$205: now also U59.6, U60.1; no longer U51.5, U52.2
- net N$206: now also U59.5, U60.2; no longer U52.6, U53.1
- net N$207: now also U6.6, U7.1; no longer U52.5, U53.2
- net N$208: now also U6.5, U7.2; no longer U54.6, U55.1
- net N$209: now also U60.6, U61.1; no longer U54.5, U55.2
- net N$210: now also U60.5, U61.2; no longer U55.6, U56.1
- net N$211: now also U62.6, U63.1; no longer U55.5, U56.2
- net N$212: now also U62.5, U63.2; no longer U56.6, U57.1
- net N$213: now also U63.6, U64.1; no longer U56.5, U57.2
- net N$214: now also U63.5, U64.2; no longer U57.6, U58.1
- net N$215: now also U64.6, U65.1; no longer U57.5, U58.2
- net N$216: no longer U58.6, U59.1
- net N$217: no longer U58.5, U59.2
- net N$218: no longer U59.6, U60.1
- net N$219: no longer U59.5, U60.2
- net N$220: no longer U6.6, U7.1
- net N$221: no longer U6.5, U7.2
- net N$222: no longer U60.6, U61.1
- net N$223: no longer U60.5, U61.2
- net N$224: no longer U62.6, U63.1
- net N$225: no longer U62.5, U63.2
- net N$226: no longer U63.6, U64.1
- net N$227: no longer U63.5, U64.2
- net N$228: no longer U64.6, U65.1
- net SQ_A1: now also U1.4; no longer U1.21
- net SQ_A2: now also U1.6; no longer U1.25
- net SQ_A3: now also U3.4; no longer U1.1
- net SQ_A4: now also U3.6; no longer U1.5
- net SQ_A5: now also U70.4; no longer U3.21
- net SQ_A6: now also U70.6; no longer U3.25
- net SQ_A7: now also U72.4; no longer U3.1
- net SQ_A8: now also U72.6; no longer U3.5
- net SQ_B1: now also U1.5; no longer U1.22
- net SQ_B2: now also U1.7; no longer U1.26
- net SQ_B3: now also U3.5; no longer U1.2
- net SQ_B4: now also U3.7; no longer U1.6
- net SQ_B5: now also U70.5; no longer U3.22
- net SQ_B6: now also U70.7; no longer U3.26
- net SQ_B7: now also U72.5; no longer U3.2
- net SQ_B8: now also U72.7; no longer U3.6
- net SQ_C1: now also U1.9; no longer U1.23
- net SQ_C2: now also U1.11; no longer U1.27
- net SQ_C3: now also U3.9; no longer U1.3
- net SQ_C4: now also U3.11; no longer U1.7
- net SQ_C5: now also U70.9; no longer U3.23
- net SQ_C6: now also U70.11; no longer U3.27
- net SQ_C7: now also U72.9; no longer U3.3
- net SQ_C8: now also U72.11; no longer U3.7
- net SQ_D1: now also U1.10; no longer U1.24
- net SQ_D2: now also U1.12; no longer U1.28
- net SQ_D3: now also U3.10; no longer U1.4
- net SQ_D4: now also U3.12; no longer U1.8
- net SQ_D5: now also U70.10; no longer U3.24
- net SQ_D6: now also U70.12; no longer U3.28
- net SQ_D7: now also U72.10; no longer U3.4
- net SQ_D8: now also U72.12; no longer U3.8
- net SQ_E1: now also U2.4; no longer U2.21
- net SQ_E2: now also U2.6; no longer U2.25
- net SQ_E3: now also U4.4; no longer U2.1
- net SQ_E4: now also U4.6; no longer U2.5
- net SQ_E5: now also U71.4; no longer U4.21
- net SQ_E6: now also U71.6; no longer U4.25
- net SQ_E7: now also U73.4; no longer U4.1
- net SQ_E8: now also U73.6; no longer U4.5
- net SQ_F1: now also U2.5; no longer U2.22
- net SQ_F2: now also U2.7; no longer U2.26
- net SQ_F3: now also U4.5; no longer U2.2
- net SQ_F4: now also U4.7; no longer U2.6
- net SQ_F5: now also U71.5; no longer U4.22
- net SQ_F6: now also U71.7; no longer U4.26
- net SQ_F7: now also U73.5; no longer U4.2
- net SQ_F8: now also U73.7; no longer U4.6
- net SQ_G1: now also U2.9; no longer U2.23
- net SQ_G2: now also U2.11; no longer U2.27
- net SQ_G3: now also U4.9; no longer U2.3
- net SQ_G4: now also U4.11; no longer U2.7
- net SQ_G5: now also U71.9; no longer U4.23
- net SQ_G6: now also U71.11; no longer U4.27
- net SQ_G7: now also U73.9; no longer U4.3
- net SQ_G8: now also U73.11; no longer U4.7
- net SQ_H1: now also U2.10; no longer U2.24
- net SQ_H2: now also U2.12; no longer U2.28
- net SQ_H3: now also U4.10; no longer U2.4
- net SQ_H4: now also U4.12; no longer U2.8
- net SQ_H5: now also U71.10; no longer U4.24
- net SQ_H6: now also U71.12; no longer U4.28
- net SQ_H7: now also U73.10; no longer U4.4
- net SQ_H8: now also U73.12; no longer U4.8
- removed net SENSE_IRQ: J1.7, U1.20, U2.20, U3.20, U4.20
- new net N$115: U10.1, U9.6
- new net N$116: U10.2, U9.5
- new net N$117: U10.6, U11.1
- new net N$118: U10.5, U11.2
- new net N$139: U23.6, U24.1
- new net N$140: U23.5, U24.2
- new net N$141: U24.6, U25.1
- new net N$158: U33.5, U34.2
- new net N$159: U34.6, U35.1
- new net N$160: U34.5, U35.2
- new net N$179: U46.6, U47.1
- new net N$180: U46.5, U47.2
- new net N$181: U47.6, U48.1
- new net N$200: U56.5, U57.2
- new net N$201: U57.6, U58.1
- no-connect marks 27 -> 24
Other:
- moved on the sheet: C14, C15, C16, C17, C18, C19, C2, C20, C21, C22, C23, C24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
