File: hardware/pcb/generated/chess-board.kicad_pcb (KiCad board)
At the start: 8 copper layers, 320 x 360 mm, 312 parts, among them J1 PPPC202LFBN-RC, J2 PPPC041LFBN-RC, J3 PJ-102A, SW1 TL1105SPF100QG, SW10 TL1105SPF100QG, SW11 TL1105SPF100QG, SW12 TL1105SPF100QG, SW13 RA11131100, SW2 TL1105SPF100QG, SW3 TL1105SPF100QG, SW4 TL1105SPF100QG, SW5 TL1105SPF100QG, SW6 TL1105SPF100QG, SW7 TL1105SPF100QG, SW8 TL1105SPF100QG, SW9 TL1105SPF100QG, U1 MCP23017-E/SO, U10 SK9822-EC20, U11 SK9822-EC20, U12 SK9822-EC20, U13 SK9822-EC20, U14 SK9822-EC20, U15 SK9822-EC20, U16 SK9822-EC20, U17 SK9822-EC20, U18 SK9822-EC20, U19 SK9822-EC20, U2 MCP23017-E/SO, U20 SK9822-EC20, U21 SK9822-EC20, U22 SK9822-EC20, U23 SK9822-EC20, U24 SK9822-EC20, U25 SK9822-EC20, U26 SK9822-EC20, U27 SK9822-EC20, U28 SK9822-EC20, U29 SK9822-EC20, U3 MCP23017-E/SO, U30 SK9822-EC20, U31 SK9822-EC20, U32 SK9822-EC20, U33 SK9822-EC20, U34 SK9822-EC20, U35 SK9822-EC20, U36 SK9822-EC20, U37 SK9822-EC20, U38 SK9822-EC20, U39 SK9822-EC20, U4 MCP23017-E/SO, U40 SK9822-EC20, U41 SK9822-EC20, U42 SK9822-EC20, U43 SK9822-EC20, U44 SK9822-EC20, U45 SK9822-EC20, U46 SK9822-EC20, U47 SK9822-EC20, U48 SK9822-EC20, U49 SK9822-EC20, U5 SN74AHCT125DR, U50 SK9822-EC20, U51 SK9822-EC20, U52 SK9822-EC20, U53 SK9822-EC20, U54 SK9822-EC20, U55 SK9822-EC20, U56 SK9822-EC20, U57 SK9822-EC20, U58 SK9822-EC20, U59 SK9822-EC20, U6 SK9822-EC20, U60 SK9822-EC20, U61 SK9822-EC20, U62 SK9822-EC20, U63 SK9822-EC20, U64 SK9822-EC20, U65 SK9822-EC20, U66 SK9822-EC20, U67 SK9822-EC20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

Commit message: fix(pcb): harden fabrication release design
Parts:
- removed the SW13 at (87.0, 410.0)
- added SW1: TL1105SPF100QG, , F.Cu at (200.0, 392.0)
- added SW2: TL1105SPF100QG, , F.Cu at (216.0, 392.0)
- added TP5: S1751-46R, , F.Cu at (181.0, 385.0)
- added TP6: S1751-46R, , F.Cu at (188.0, 385.0)
- added TP7: S1751-46R, , F.Cu at (153.0, 416.0)
- added TP8: S1751-46R, , F.Cu at (160.0, 416.0)
- F1: value 0453005.MR -> 0453002.MR
- R3: renamed from SW1; value TL1105SPF100QG -> RC0603FR-074K7L
- SW13: renamed from SW2; value TL1105SPF100QG -> RA11131100
- moved SW13 130.2 mm to (87.0, 410.0)
- moved R3 19.0 mm to (181.0, 393.0)
- moved TP1 7.00 mm to (153.0, 385.0)
- moved TP2 7.00 mm to (160.0, 385.0)
- moved TP3 7.00 mm to (167.0, 385.0)
- moved TP4 7.00 mm to (174.0, 385.0)
- turned J3 to -90 degrees
Connections:
- R3 pad 1: BTN_UP -> +3V3
- R3 pad 2: GND -> SENSE_IRQ
- SW13 pad 1: BTN_DOWN -> DC_FUSED
- SW13 pad 2: GND -> +5V
Routing:
- net SENSE_IRQ: track 624.7 -> 725.5 mm, vias 4 -> 6
- net I2C_SDA: track 703.1 -> 733.4 mm, vias 9 -> 10
- net I2C_SCL: track 742.5 -> 762.5 mm, vias 6 -> 7
- net LED_CLK_5V: track 193.9 -> 186.9 mm
- net LED_DATA_5V: track 181.9 -> 174.9 mm
- net SQ_D1: track 87.1 -> 91.0 mm, vias 2 -> 3
- net DC_IN: track 23.2 -> 21.7 mm
- net +3V3: track 91.6 -> 92.0 mm, vias 146 -> 148
Other:
- board text added: "3V3"
- board text added: "5V"
- board text added: "CHESS BOARD C-PROTOTYPE"
- board text added: "CLK"
- board text added: "D1 K=+5V"
- board text added: "DATA"
- board text added: "DOWN"
- board text added: "F1"
- board text added: "F1 2A MAX"
- board text added: "F2"
- board text added: "F3"
- board text added: "F4"
- board text added: "F5"
- board text added: "GND"
- board text added: "IRQ"
- board text added: "J2: GND 3V3 SCL SDA"
- board text added: "J3 5V CENTER +"
- board text added: "LEFT"
- board text added: "OK"
- board text added: "PASS"
- board text added: "RESET"
- board text added: "RIGHT"
- board text added: "SCL"
- board text added: "SDA"
- board text added: "SW13 POWER"
- board text added: "UP"

Commit message: Add PCB connection silkscreen labels
Other:
- board text added: "16 F4 18 F5 19 SPI-DATA 23 SPI-CLK"
- board text added: "29 UP 31 DOWN 32 LEFT 33 RIGHT 35 PASS 36 OK"
- board text added: "38 F1 40 F2 | 1/17 3V3 | 2/4 5V | GND: 6/9/14/20/25/30/34/39"
- board text added: "A1"
- board text added: "A2"
- board text added: "A3"
- board text added: "A4"
- board text added: "A5"
- board text added: "A6"
- board text added: "A7"
- board text added: "A8"
- board text added: "B1"
- board text added: "B2"
- board text added: "B3"
- board text added: "B4"
- board text added: "B5"
- board text added: "B6"
- board text added: "B7"
- board text added: "B8"
- board text added: "C1"
- board text added: "C2"
- board text added: "C3"
- board text added: "C4"
- board text added: "C5"
- board text added: "C6"
- board text added: "C7"
- board text added: "C8"
- board text added: "D1"
- board text added: "D2"
- board text added: "D3"
- board text added: "D4"
- board text added: "D5"
- board text added: "D6"
- board text added: "D7"
- board text added: "D8"
- board text added: "E1"
- board text added: "E2"
- board text added: "E3"
- board text added: "E4"
- board text added: "E5"
- board text added: "E6"
- board text added: "E7"
- board text added: "E8"
- board text added: "F6"
- board text added: "F7"
- board text added: "F8"
- board text added: "G1"
- board text added: "G2"
- board text added: "G3"
- board text added: "G4"
- board text added: "G5"
- board text added: "G6"
- board text added: "G7"
- board text added: "G8"
- board text added: "H1"
- board text added: "H2"
- board text added: "H3"
- board text added: "H4"
- board text added: "H5"
- board text added: "H6"
- board text added: "H7"
- board text added: "H8"
- board text added: "J1 PI: 3 SDA 5 SCL 7 IRQ 11 RESET 15 F3"
- board text added: "LED CHAIN END"
- board text added: "LED DATA + CLK IN"
- board text added: "R1/R2 I2C PULL-UPS"
- board text added: "R3 IRQ PULL-UP"
- board text added: "U1 I2C 0x20 A1-D4"
- board text added: "U2 I2C 0x21 E1-H4"
- board text added: "U3 I2C 0x22 A5-D8"
- board text added: "U4 I2C 0x23 E5-H8"
- board text added: "U5 SPI 3V3 -> LED 5V"
