File: hardware/pcb/generated/chess-board.kicad_pcb (KiCad board)
At the start: 8 copper layers, 320 x 360 mm, 317 parts, among them J1 PPPC202LFBN-RC, J2 PPPC041LFBN-RC, J3 PJ-102A, SW1 TL1105SPF100QG, SW10 TL1105SPF100QG, SW11 TL1105SPF100QG, SW12 TL1105SPF100QG, SW13 RA11131100, SW2 TL1105SPF100QG, SW3 TL1105SPF100QG, SW4 TL1105SPF100QG, SW5 TL1105SPF100QG, SW6 TL1105SPF100QG, SW7 TL1105SPF100QG, SW8 TL1105SPF100QG, SW9 TL1105SPF100QG, U1 MCP23017-E/SO, U10 SK9822-EC20, U11 SK9822-EC20, U12 SK9822-EC20, U13 SK9822-EC20, U14 SK9822-EC20, U15 SK9822-EC20, U16 SK9822-EC20, U17 SK9822-EC20, U18 SK9822-EC20, U19 SK9822-EC20, U2 MCP23017-E/SO, U20 SK9822-EC20, U21 SK9822-EC20, U22 SK9822-EC20, U23 SK9822-EC20, U24 SK9822-EC20, U25 SK9822-EC20, U26 SK9822-EC20, U27 SK9822-EC20, U28 SK9822-EC20, U29 SK9822-EC20, U3 MCP23017-E/SO, U30 SK9822-EC20, U31 SK9822-EC20, U32 SK9822-EC20, U33 SK9822-EC20, U34 SK9822-EC20, U35 SK9822-EC20, U36 SK9822-EC20, U37 SK9822-EC20, U38 SK9822-EC20, U39 SK9822-EC20, U4 MCP23017-E/SO, U40 SK9822-EC20, U41 SK9822-EC20, U42 SK9822-EC20, U43 SK9822-EC20, U44 SK9822-EC20, U45 SK9822-EC20, U46 SK9822-EC20, U47 SK9822-EC20, U48 SK9822-EC20, U49 SK9822-EC20, U5 SN74AHCT125DR, U50 SK9822-EC20, U51 SK9822-EC20, U52 SK9822-EC20, U53 SK9822-EC20, U54 SK9822-EC20, U55 SK9822-EC20, U56 SK9822-EC20, U57 SK9822-EC20, U58 SK9822-EC20, U59 SK9822-EC20, U6 SK9822-EC20, U60 SK9822-EC20, U61 SK9822-EC20, U62 SK9822-EC20, U63 SK9822-EC20, U64 SK9822-EC20, U65 SK9822-EC20, U66 SK9822-EC20, U67 SK9822-EC20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

Commit message: Standardize PCB routing coordinates
Routing:
- net N$130: track 76.6 -> 166.6 mm
- net N$129: track 71.6 -> 92.1 mm, vias 0 -> 2
- net SQ_H4: track 110.7 -> 124.0 mm
- net I2C_SCL: track 762.5 -> 750.5 mm, vias 7 -> 9
- net N$137: track 109.6 -> 119.6 mm, vias 0 -> 2
- net SQ_G4: track 70.8 -> 80.3 mm
- net SQ_F4: track 86.0 -> 76.9 mm
- net SENSE_IRQ: track 725.5 -> 718.5 mm
- net GND: track 154.8 -> 149.2 mm
- net +5V: track 61.6 -> 56.0 mm
- net SQ_F2: track 64.1 -> 69.4 mm, vias 2 -> 0
- net SQ_G1: track 77.2 -> 74.3 mm
- net SQ_F1: track 90.6 -> 88.2 mm
- net I2C_SDA: track 733.4 -> 732.4 mm
- net SQ_G2: track 40.5 -> 39.9 mm, vias 2 -> 0
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