File: hardware/pcb/generated/chess-board.kicad_pcb (KiCad board)
At the start: 8 copper layers, 320 x 360 mm, 317 parts, among them J1 PPPC202LFBN-RC, J2 PPPC041LFBN-RC, J3 PJ-102A, SW1 TL1105SPF100QG, SW10 TL1105SPF100QG, SW11 TL1105SPF100QG, SW12 TL1105SPF100QG, SW13 RA11131100, SW2 TL1105SPF100QG, SW3 TL1105SPF100QG, SW4 TL1105SPF100QG, SW5 TL1105SPF100QG, SW6 TL1105SPF100QG, SW7 TL1105SPF100QG, SW8 TL1105SPF100QG, SW9 TL1105SPF100QG, U1 MCP23017-E/SO, U10 SK9822-EC20, U11 SK9822-EC20, U12 SK9822-EC20, U13 SK9822-EC20, U14 SK9822-EC20, U15 SK9822-EC20, U16 SK9822-EC20, U17 SK9822-EC20, U18 SK9822-EC20, U19 SK9822-EC20, U2 MCP23017-E/SO, U20 SK9822-EC20, U21 SK9822-EC20, U22 SK9822-EC20, U23 SK9822-EC20, U24 SK9822-EC20, U25 SK9822-EC20, U26 SK9822-EC20, U27 SK9822-EC20, U28 SK9822-EC20, U29 SK9822-EC20, U3 MCP23017-E/SO, U30 SK9822-EC20, U31 SK9822-EC20, U32 SK9822-EC20, U33 SK9822-EC20, U34 SK9822-EC20, U35 SK9822-EC20, U36 SK9822-EC20, U37 SK9822-EC20, U38 SK9822-EC20, U39 SK9822-EC20, U4 MCP23017-E/SO, U40 SK9822-EC20, U41 SK9822-EC20, U42 SK9822-EC20, U43 SK9822-EC20, U44 SK9822-EC20, U45 SK9822-EC20, U46 SK9822-EC20, U47 SK9822-EC20, U48 SK9822-EC20, U49 SK9822-EC20, U5 SN74AHCT125DR, U50 SK9822-EC20, U51 SK9822-EC20, U52 SK9822-EC20, U53 SK9822-EC20, U54 SK9822-EC20, U55 SK9822-EC20, U56 SK9822-EC20, U57 SK9822-EC20, U58 SK9822-EC20, U59 SK9822-EC20, U6 SK9822-EC20, U60 SK9822-EC20, U61 SK9822-EC20, U62 SK9822-EC20, U63 SK9822-EC20, U64 SK9822-EC20, U65 SK9822-EC20, U66 SK9822-EC20, U67 SK9822-EC20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

Commit message: chore(hardware): refresh PCB and firmware outputs
Parts:
- removed R3: RC0603FR-074K7L, 
- removed TP8: S1751-46R, 
- removed the U9 at (193.0, 347.0)
- added C136: CC0603KRX7R9BB104, , F.Cu at (128.0, 172.0)
- added C137: CC0603KRX7R9BB104, , F.Cu at (288.0, 172.0)
- added C138: CC0603KRX7R9BB104, , F.Cu at (128.0, 92.0)
- added C139: CC0603KRX7R9BB104, , F.Cu at (288.0, 92.0)
- added H8: M3 mounting hole, , F.Cu at (320.0, 260.0)
- added U70: TCA9554DWR, , F.Cu at (120.0, 178.0)
- added U71: TCA9554DWR, , F.Cu at (280.0, 178.0)
- added U72: TCA9554DWR, , F.Cu at (120.0, 98.0)
- added U73: TCA9554DWR, , F.Cu at (280.0, 98.0)
- U1, U2, U3, U4: value MCP23017-E/SO -> TCA9554DWR
- U9: renamed from H8; value M3 mounting hole -> SK9822-EC20
- moved U9 153.9 mm to (193.0, 347.0)
- moved U3 118.8 mm to (120.0, 258.0)
- moved U4 118.8 mm to (280.0, 258.0)
- moved C5 100.2 mm to (128.0, 252.0)
- moved C6 100.2 mm to (288.0, 252.0)
- moved U1 40.5 mm to (120.0, 338.0)
- moved U2 40.5 mm to (280.0, 338.0)
- moved C3 20.9 mm to (128.0, 332.0)
- moved C4 20.9 mm to (288.0, 332.0)
Connections:
- J1 pad 7: SENSE_IRQ -> unconnected-(J1-Pad7)
- U1 pad 1: SQ_A3 -> GND
- U1 pad 10: GND -> SQ_D1
- U1 pad 11: unconnected-(U1-Pad11) -> SQ_C2
- U1 pad 12: I2C_SCL -> SQ_D2
- U1 pad 13: I2C_SDA -> unconnected-(U1-Pad13)
- U1 pad 14: unconnected-(U1-Pad14) -> I2C_SCL
- U1 pad 15: GND -> I2C_SDA
- U1 pad 16: GND -> +3V3
- U1 pad 2: SQ_B3 -> GND
- U1 pad 3: SQ_C3 -> GND
- U1 pad 4: SQ_D3 -> SQ_A1
- U1 pad 5: SQ_A4 -> SQ_B1
- U1 pad 6: SQ_B4 -> SQ_A2
- U1 pad 7: SQ_C4 -> SQ_B2
- U1 pad 8: SQ_D4 -> GND
- U1 pad 9: +3V3 -> SQ_C1
- U10 pad 1: N$119 (its old number) -> N$115
- U10 pad 2: N$120 (its old number) -> N$116
- U2 pad 1: SQ_E3 -> +3V3
- U2 pad 10: GND -> SQ_H1
- U2 pad 11: unconnected-(U2-Pad11) -> SQ_G2
- U2 pad 12: I2C_SCL -> SQ_H2
- U2 pad 13: I2C_SDA -> unconnected-(U2-Pad13)
- U2 pad 14: unconnected-(U2-Pad14) -> I2C_SCL
- U2 pad 15: +3V3 -> I2C_SDA
- U2 pad 16: GND -> +3V3
- U2 pad 2: SQ_F3 -> GND
- U2 pad 3: SQ_G3 -> GND
- U2 pad 4: SQ_H3 -> SQ_E1
- U2 pad 5: SQ_E4 -> SQ_F1
- U2 pad 6: SQ_F4 -> SQ_E2
- U2 pad 7: SQ_G4 -> SQ_F2
- U2 pad 8: SQ_H4 -> GND
- U2 pad 9: +3V3 -> SQ_G1
- U3 pad 1: SQ_A7 -> GND
- U3 pad 10: GND -> SQ_D3
- U3 pad 11: unconnected-(U3-Pad11) -> SQ_C4
- U3 pad 12: I2C_SCL -> SQ_D4
- U3 pad 13: I2C_SDA -> unconnected-(U3-Pad13)
- U3 pad 14: unconnected-(U3-Pad14) -> I2C_SCL
- U3 pad 15: GND -> I2C_SDA
- U3 pad 2: SQ_B7 -> +3V3
- U3 pad 3: SQ_C7 -> GND
- U3 pad 4: SQ_D7 -> SQ_A3
- U3 pad 5: SQ_A8 -> SQ_B3
- U3 pad 6: SQ_B8 -> SQ_A4
- U3 pad 7: SQ_C8 -> SQ_B4
- U3 pad 8: SQ_D8 -> GND
- U3 pad 9: +3V3 -> SQ_C3
- U4 pad 1: SQ_E7 -> +3V3
- U4 pad 10: GND -> SQ_H3
- U4 pad 11: unconnected-(U4-Pad11) -> SQ_G4
- U4 pad 12: I2C_SCL -> SQ_H4
- U4 pad 13: I2C_SDA -> unconnected-(U4-Pad13)
- U4 pad 14: unconnected-(U4-Pad14) -> I2C_SCL
- U4 pad 15: +3V3 -> I2C_SDA
- U4 pad 2: SQ_F7 -> +3V3
- U4 pad 3: SQ_G7 -> GND
- U4 pad 4: SQ_H7 -> SQ_E3
- U4 pad 5: SQ_E8 -> SQ_F3
- U4 pad 6: SQ_F8 -> SQ_E4
- U4 pad 7: SQ_G8 -> SQ_F4
- U4 pad 8: SQ_H8 -> GND
- U4 pad 9: +3V3 -> SQ_G3
- U8 pad 5: N$241 -> N$228
- U8 pad 6: N$240 -> N$227
Routing:
- net SENSE_IRQ: track 718.5 -> 0.00 mm, vias 6 -> 0
- net I2C_SDA: track 732.4 -> 887.8 mm, vias 10 -> 14
- net I2C_SCL: track 750.5 -> 893.6 mm, vias 9 -> 11
- net N$126: track 166.6 -> 35.0 mm, vias 4 -> 0
- net N$134: track 134.1 -> 35.0 mm
- net N$133: track 119.6 -> 35.0 mm, vias 2 -> 0
- net SQ_D4: track 124.0 -> 61.8 mm, vias 3 -> 2
- net SQ_H4: track 124.0 -> 61.8 mm, vias 3 -> 2
- net N$125: track 92.1 -> 35.0 mm, vias 2 -> 0
- net SQ_B5: track 92.3 -> 36.6 mm
- net SQ_C5: track 82.2 -> 27.5 mm
- net SQ_G5: track 82.2 -> 27.5 mm
- net SQ_E1: track 130.7 -> 77.1 mm, vias 2 -> 4
- net N$192: track 88.1 -> 35.0 mm, vias 2 -> 0
- net N$182: track 88.1 -> 35.0 mm, vias 2 -> 0
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Other:
- board text added: "CHESS BOARD D-PROTOTYPE"
- board text added: "J1 PI: 3 SDA 5 SCL 11 RESET 15 F3"
- board text added: "U1 I2C 0x20 A1-D2"
- board text added: "U2 I2C 0x21 E1-H2"
- board text added: "U3 I2C 0x22 A3-D4"
- board text added: "U4 I2C 0x23 E3-H4"
- board text added: "U70 I2C 0x24 A5-D6"
- board text added: "U71 I2C 0x25 E5-H6"
- board text added: "U72 I2C 0x26 A7-D8"
- board text added: "U73 I2C 0x27 E7-H8"
- board text removed: "CHESS BOARD C-PROTOTYPE"
- board text removed: "IRQ"
- board text removed: "J1 PI: 3 SDA 5 SCL 7 IRQ 11 RESET 15 F3"
- board text removed: "R3 IRQ PULL-UP"
- board text removed: "U1 I2C 0x20 A1-D4"
- board text removed: "U2 I2C 0x21 E1-H4"
- board text removed: "U3 I2C 0x22 A5-D8"
- board text removed: "U4 I2C 0x23 E5-H8"
