File: hardware/pcb/generated/bank-A5-D6.kicad_sch (KiCad schematic)
At the start: 34 parts, among them U38 SK9822-EC20, U39 SK9822-EC20, U40 SK9822-EC20, U41 SK9822-EC20, U50 SK9822-EC20, U51 SK9822-EC20, U52 SK9822-EC20, U53 SK9822-EC20, U70 TCA9554DWR

Commit message: chore(pcb): regenerate KiCad, SPICE and review output
Generated by `just pcb` from the committed definition; not hand-edited.
Parts:
- U38, U39, U40, U41, U50, U51, U52, U53: value SK9822-EC20 -> SK9822-A
Connections:
- net +5V renamed LED_5V
- net LED_D48 renamed LED_D48_SRC
