File: hardware/pcb/generated/bank-E5-H6.kicad_sch (KiCad schematic)
At the start: 34 parts, among them U42 SK9822-EC20, U43 SK9822-EC20, U44 SK9822-EC20, U45 SK9822-EC20, U46 SK9822-EC20, U47 SK9822-EC20, U48 SK9822-EC20, U49 SK9822-EC20, U71 TCA9554DWR

Commit message: chore(pcb): regenerate KiCad, SPICE and review output
Generated by `just pcb` from the committed definition; not hand-edited.
Parts:
- U42, U43, U44, U45, U46, U47, U48, U49: value SK9822-EC20 -> SK9822-A
Connections:
- net +5V renamed LED_5V
