File: hardware/pcb/generated/components-01.kicad_sch (KiCad schematic)
At the start: 12 parts

Commit message: refactor: unify PCB and CAD generation with verified models
Parts:
- C1: footprint (none) -> CAP_560U
- C10, C100, C101, C102, C103, C104, C105, C106, C107, C108, C109: footprint (none) -> CAP_100N
