File: hardware/pcb/generated/components-02.kicad_sch (KiCad schematic)
At the start: 12 parts

Commit message: refactor: unify PCB and CAD generation with verified models
Parts:
- C11, C110, C111, C112, C113, C114, C115, C116, C117, C118, C119, C12: footprint (none) -> CAP_100N
