File: hardware/pcb/generated/components-03.kicad_sch (KiCad schematic)
At the start: 12 parts

Commit message: refactor: unify PCB and CAD generation with verified models
Parts:
- C120, C121, C122, C123, C124, C125, C126, C127, C128, C129, C13, C130: footprint (none) -> CAP_100N
