File: hardware/pcb/generated/components-04.kicad_sch (KiCad schematic)
At the start: 12 parts

Commit message: refactor: unify PCB and CAD generation with verified models
Parts:
- C131, C132, C133, C134, C135, C136, C137, C138, C139, C14: footprint (none) -> CAP_100N
- C140: footprint (none) -> CAP_560U
- C141: footprint (none) -> CAP_1U
