File: hardware/pcb/generated/components-05.kicad_sch (KiCad schematic)
At the start: 12 parts

Commit message: refactor: unify PCB and CAD generation with verified models
Parts:
- C142, C144, C145: footprint (none) -> CAP_10N
- C143: footprint (none) -> CAP_1N
- C146, C15, C16, C17, C18, C19, C20: footprint (none) -> CAP_100N
- C2: footprint (none) -> CAP_10U
