File: hardware/pcb/generated/components-06.kicad_sch (KiCad schematic)
At the start: 12 parts

Commit message: refactor: unify PCB and CAD generation with verified models
Parts:
- C21, C22, C23, C24, C25, C26, C27, C28, C29, C3, C30, C31: footprint (none) -> CAP_100N
