File: hardware/pcb/generated/components-07.kicad_sch (KiCad schematic)
At the start: 12 parts

Commit message: refactor: unify PCB and CAD generation with verified models
Parts:
- C32, C33, C34, C35, C36, C37, C38, C39, C4, C40, C41, C42: footprint (none) -> CAP_100N
