File: hardware/pcb/generated/components-08.kicad_sch (KiCad schematic)
At the start: 12 parts

Commit message: refactor: unify PCB and CAD generation with verified models
Parts:
- C43, C44, C45, C46, C47, C48, C49, C5, C50, C51, C52, C53: footprint (none) -> CAP_100N
