File: hardware/pcb/generated/components-09.kicad_sch (KiCad schematic)
At the start: 12 parts

Commit message: refactor: unify PCB and CAD generation with verified models
Parts:
- C54, C55, C56, C57, C58, C59, C6, C60, C61, C62, C63, C64: footprint (none) -> CAP_100N
