File: hardware/pcb/generated/components-10.kicad_sch (KiCad schematic)
At the start: 12 parts

Commit message: refactor: unify PCB and CAD generation with verified models
Parts:
- C65, C66, C67, C68, C69, C7, C70, C71, C72, C73, C74, C75: footprint (none) -> CAP_100N
