File: hardware/pcb/generated/components-11.kicad_sch (KiCad schematic)
At the start: 12 parts

Commit message: refactor: unify PCB and CAD generation with verified models
Parts:
- C76, C77, C78, C79, C8, C80, C81, C82, C83, C84, C85, C86: footprint (none) -> CAP_100N
