File: hardware/pcb/generated/components-12.kicad_sch (KiCad schematic)
At the start: 12 parts

Commit message: refactor: unify PCB and CAD generation with verified models
Parts:
- C87, C88, C89, C9, C90, C91, C92, C93, C94, C95, C96, C97: footprint (none) -> CAP_100N
