File: hardware/pcb/generated/components-13.kicad_sch (KiCad schematic)
At the start: 12 parts

Commit message: refactor: unify PCB and CAD generation with verified models
Parts:
- C98, C99: footprint (none) -> CAP_100N
- D1: footprint (none) -> TVS_12V0
- F1: footprint (none) -> FUSE_2A
- HS1, HS10, HS11, HS12, HS13, HS14, HS15, HS16: footprint (none) -> HALL_SENSOR
