File: hardware/pcb/generated/components-14.kicad_sch (KiCad schematic)
At the start: 12 parts

Commit message: refactor: unify PCB and CAD generation with verified models
Parts:
- HS17, HS18, HS19, HS2, HS20, HS21, HS22, HS23, HS24, HS25, HS26, HS27: footprint (none) -> HALL_SENSOR
