File: hardware/pcb/generated/components-15.kicad_sch (KiCad schematic)
At the start: 12 parts

Commit message: refactor: unify PCB and CAD generation with verified models
Parts:
- HS28, HS29, HS3, HS30, HS31, HS32, HS33, HS34, HS35, HS36, HS37, HS38: footprint (none) -> HALL_SENSOR
