File: hardware/pcb/generated/components-16.kicad_sch (KiCad schematic)
At the start: 12 parts

Commit message: refactor: unify PCB and CAD generation with verified models
Parts:
- HS39, HS4, HS40, HS41, HS42, HS43, HS44, HS45, HS46, HS47, HS48, HS49: footprint (none) -> HALL_SENSOR
