File: hardware/pcb/generated/components-17.kicad_sch (KiCad schematic)
At the start: 12 parts

Commit message: refactor: unify PCB and CAD generation with verified models
Parts:
- HS5, HS50, HS51, HS52, HS53, HS54, HS55, HS56, HS57, HS58, HS59, HS6: footprint (none) -> HALL_SENSOR
