File: hardware/pcb/generated/components-18.kicad_sch (KiCad schematic)
At the start: 12 parts, among them J1 PPPC202LFBN-RC, J2 SM04B-SRSS-TB, J4 B4PS-VH, Q1 Si4403DDY-T1-GE3

Commit message: refactor: unify PCB and CAD generation with verified models
Parts:
- HS60, HS61, HS62, HS63, HS64, HS7, HS8, HS9: footprint (none) -> HALL_SENSOR
- J1: footprint (none) -> PI_ZERO_HEADER
- J2: footprint (none) -> OLED_HEADER
- J4: footprint (none) -> POWER_HEADER
- Q1: footprint (none) -> LED_SWITCH
