File: hardware/pcb/generated/components-19.kicad_sch (KiCad schematic)
At the start: 12 parts, among them Q2 BSS138LT1G

Commit message: refactor: unify PCB and CAD generation with verified models
Parts:
- Q2: footprint (none) -> LED_SWITCH_DRIVER
- R10, R11, R12: footprint (none) -> RES_56
- R13: footprint (none) -> RES_1K
- R14, R16: footprint (none) -> RES_100K
- R15, R17, R18: footprint (none) -> RES_10K
- R3: footprint (none) -> RES_1K65
- R4: footprint (none) -> RES_604K_PRECISION
