File: hardware/pcb/generated/components-20.kicad_sch (KiCad schematic)
At the start: 12 parts, among them SW1 TL1105CF100Q, SW10 TL1105CF100Q, SW11 TL1105CF100Q, SW12 TL1105CF100Q, SW2 TL1105CF100Q, SW3 TL1105CF100Q, SW4 TL1105CF100Q

Commit message: refactor: unify PCB and CAD generation with verified models
Parts:
- R5: footprint (none) -> RES_169K_PRECISION
- R6: footprint (none) -> RES_604K_PRECISION
- R7: footprint (none) -> RES_261K
- R8: footprint (none) -> RES_1K
- R9: footprint (none) -> RES_56
- SW1, SW10, SW11, SW12, SW2, SW3, SW4: footprint (none) -> BUTTON
