File: hardware/pcb/generated/components-21.kicad_sch (KiCad schematic)
At the start: 12 parts, among them SW5 TL1105CF100Q, SW6 TL1105CF100Q, SW7 TL1105CF100Q, SW8 TL1105CF100Q, SW9 TL1105CF100Q

Commit message: refactor: unify PCB and CAD generation with verified models
Parts:
- SW5, SW6, SW7, SW8, SW9: footprint (none) -> BUTTON
- TP1, TP2, TP3, TP4, TP5, TP6, TP7: footprint (none) -> TEST_POINT
