File: hardware/pcb/generated/components-22.kicad_sch (KiCad schematic)
At the start: 12 parts, among them U1 TCA9554DWR, U10 SK9822-A, U11 SK9822-A, U12 SK9822-A, U13 SK9822-A, U14 SK9822-A, U15 SK9822-A, U16 SK9822-A, U17 SK9822-A, U18 SK9822-A, U19 SK9822-A, U2 TCA9554DWR

Commit message: refactor: unify PCB and CAD generation with verified models
Parts:
- U1, U2: footprint (none) -> TCA9554
- U10, U11, U12, U13, U14, U15, U16, U17, U18, U19: footprint (none) -> SK9822
