File: hardware/pcb/generated/components-23.kicad_sch (KiCad schematic)
At the start: 12 parts, among them U20 SK9822-A, U21 SK9822-A, U22 SK9822-A, U23 SK9822-A, U24 SK9822-A, U25 SK9822-A, U26 SK9822-A, U27 SK9822-A, U28 SK9822-A, U29 SK9822-A, U3 TCA9554DWR, U30 SK9822-A

Commit message: refactor: unify PCB and CAD generation with verified models
Parts:
- U20, U21, U22, U23, U24, U25, U26, U27, U28, U29, U30: footprint (none) -> SK9822
- U3: footprint (none) -> TCA9554
