File: hardware/pcb/generated/components-24.kicad_sch (KiCad schematic)
At the start: 12 parts, among them U31 SK9822-A, U32 SK9822-A, U33 SK9822-A, U34 SK9822-A, U35 SK9822-A, U36 SK9822-A, U37 SK9822-A, U38 SK9822-A, U39 SK9822-A, U4 TCA9554DWR, U40 SK9822-A, U41 SK9822-A

Commit message: refactor: unify PCB and CAD generation with verified models
Parts:
- U31, U32, U33, U34, U35, U36, U37, U38, U39, U40, U41: footprint (none) -> SK9822
- U4: footprint (none) -> TCA9554
