File: hardware/pcb/generated/components-25.kicad_sch (KiCad schematic)
At the start: 12 parts, among them U42 SK9822-A, U43 SK9822-A, U44 SK9822-A, U45 SK9822-A, U46 SK9822-A, U47 SK9822-A, U48 SK9822-A, U49 SK9822-A, U5 SN74AHCT125DR, U50 SK9822-A, U51 SK9822-A, U52 SK9822-A

Commit message: refactor: unify PCB and CAD generation with verified models
Parts:
- U42, U43, U44, U45, U46, U47, U48, U49, U50, U51, U52: footprint (none) -> SK9822
- U5: footprint (none) -> AHCT125
