File: hardware/pcb/generated/components-26.kicad_sch (KiCad schematic)
At the start: 12 parts, among them U53 SK9822-A, U54 SK9822-A, U55 SK9822-A, U56 SK9822-A, U57 SK9822-A, U58 SK9822-A, U59 SK9822-A, U6 SK9822-A, U60 SK9822-A, U61 SK9822-A, U62 SK9822-A, U63 SK9822-A

Commit message: refactor: unify PCB and CAD generation with verified models
Parts:
- U53, U54, U55, U56, U57, U58, U59, U6, U60, U61, U62, U63: footprint (none) -> SK9822
