File: hardware/pcb/generated/components-27.kicad_sch (KiCad schematic)
At the start: 12 parts, among them U64 SK9822-A, U65 SK9822-A, U66 SK9822-A, U67 SK9822-A, U68 SK9822-A, U69 SK9822-A, U7 SK9822-A, U70 TCA9554DWR, U71 TCA9554DWR, U72 TCA9554DWR, U73 TCA9554DWR, U74 TPS259474ARPWR

Commit message: refactor: unify PCB and CAD generation with verified models
Parts:
- U64, U65, U66, U67, U68, U69, U7: footprint (none) -> SK9822
- U70, U71, U72, U73: footprint (none) -> TCA9554
- U74: footprint (none) -> EFUSE
