File: hardware/pcb/generated/components-28.kicad_sch (KiCad schematic)
At the start: 3 parts, among them U75 SN74LVC1G97DBVR, U8 SK9822-A, U9 SK9822-A

Commit message: refactor: unify PCB and CAD generation with verified models
Parts:
- U75: footprint (none) -> LED_ENABLE_GATE
- U8, U9: footprint (none) -> SK9822
Changed lines of the file:
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@@
 (kicad_sch (version 20250114) (generator "chess_harness") (paper "User" 420 210) (title_block (title "Components 28: U75 to U9"))
-(symbol (lib_id "Board:LED_ENABLE_GATE") (at 76.2 25.4 0) (unit 1) (in_bom yes) (on_board yes) (dnp no) (property "Reference" "U75" (at 76.2 20.32 0) (effects (font (size 1.27 1.27)))) (property "Value" "SN74LVC1G97DBVR" (at 76.2 22.86 0) (effects (font (size 1.27 1.27)))) (property "Footprint" "" (at 76.2 25.4 0) (effects (font (size 1.27 1.27)) (hide yes))) (property "Datasheet" "https://www.ti.com/lit/ds/symlink/sn74lvc1g97.pdf" (at 76.2 27.94 0) (effects (font (size 1.27 1.27)) (hide yes))) (property "Description" "LED_OE_N = Schmitt(Q1 gate) OR LED_EN_N: buffer on only once LED_5V is up" (at 76.2 30.48 0) (effects (font (size 1.27 1.27)) (hide yes))) (instances (project "chess-board" (path "/78e160a7-634d-5fb3-901f-997b418a9dc6/b595d5f5-7ddb-5b0e-9c84-e831702cdbbb" (reference "U75") (unit 1)))))
+(symbol (lib_id "Board:LED_ENABLE_GATE") (at 76.2 25.4 0) (unit 1) (in_bom yes) (on_board yes) (dnp no) (property "Reference" "U75" (at 76.2 20.32 0) (effects (font (size 1.27 1.27)))) (property "Value" "SN74LVC1G97DBVR" (at 76.2 22.86 0) (effects (font (size 1.27 1.27)))) (property "Footprint" "LED_ENABLE_GATE" (at 76.2 25.4 0) (effects (font (size 1.27 1.27)) (hide yes))) (property "Datasheet" "https://www.ti.com/lit/ds/symlink/sn74lvc1g97.pdf" (at 76.2 27.94 0) (effects (font (size 1.27 1.27)) (hide yes))) (property "Description" "LED_OE_N = Schmitt(Q1 gate) OR LED_EN_N: buffer on only once LED_5V is up" (at 76.2 30.48 0) (effects (font (size 1.27 1.27)) (hide yes))) (instances (project "chess-board" (path "/78e160a7-634d-5fb3-901f-997b418a9dc6/b595d5f5-7ddb-5b0e-9c84-e831702cdbbb" (reference "U75") (unit 1)))))
 (global_label "LED_OE_N" (shape passive) (at 53.34 27.94 0) (effects (font (size 1.016 1.016)) (justify right)))
 (global_label "+5V" (shape passive) (at 53.34 30.48 0) (effects (font (size 1.016 1.016)) (justify right)))
@@
 (global_label "GND" (shape passive) (at 53.34 38.1 0) (effects (font (size 1.016 1.016)) (justify right)))
 (global_label "LED_EN_N" (shape passive) (at 53.34 40.64 0) (effects (font (size 1.016 1.016)) (justify right)))
-(symbol (lib_id "Board:SK9822") (at 203.2 25.4 0) (unit 1) (in_bom yes) (on_board yes) (dnp no) (property "Reference" "U8" (at 203.2 20.32 0) (effects (font (size 1.27 1.27)))) (property "Value" "SK9822-A" (at 203.2 22.86 0) (effects (font (size 1.27 1.27)))) (property "Footprint" "" (at 203.2 25.4 0) (effects (font (size 1.27 1.27)) (hide yes))) (property "Datasheet" "https://www.rose-lighting.com/wp-content/uploads/sites/53/2020/05/SK9822-A-REV.01-EN-5050-RGB-27K-HZ-PWM-30M-bps-speed.pdf" (at 203.2 27.94 0) (effects (font (size 1.27 1.27)) (hide yes))) (property "Description" "Clocked 5050 RGB LED" (at 203.2 30.48 0) (effects (font (size 1.27 1.27)) (hide yes))) (instances (project "chess-board" (path "/78e160a7-634d-5fb3-901f-997b418a9dc6/b595d5f5-7ddb-5b0e-9c84-e831702cdbbb" (reference "U8") (unit 1)))))
+(symbol (lib_id "Board:SK9822") (at 203.2 25.4 0) (unit 1) (in_bom yes) (on_board yes) (dnp no) (property "Reference" "U8" (at 203.2 20.32 0) (effects (font (size 1.27 1.27)))) (property "Value" "SK9822-A" (at 203.2 22.86 0) (effects (font (size 1.27 1.27)))) (property "Footprint" "SK9822" (at 203.2 25.4 0) (effects (font (size 1.27 1.27)) (hide yes))) (property "Datasheet" "https://www.rose-lighting.com/wp-content/uploads/sites/53/2020/05/SK9822-A-REV.01-EN-5050-RGB-27K-HZ-PWM-30M-bps-speed.pdf" (at 203.2 27.94 0) (effects (font (size 1.27 1.27)) (hide yes))) (property "Description" "Clocked 5050 RGB LED" (at 203.2 30.48 0) (effects (font (size 1.27 1.27)) (hide yes))) (instances (project "chess-board" (path "/78e160a7-634d-5fb3-901f-997b418a9dc6/b595d5f5-7ddb-5b0e-9c84-e831702cdbbb" (reference "U8") (unit 1)))))
 (global_label "LED_DATA_C1_TO_D1" (shape passive) (at 180.34 27.94 0) (effects (font (size 1.016 1.016)) (justify right)))
 (global_label "LED_CLOCK_C1_TO_D1" (shape passive) (at 180.34 30.48 0) (effects (font (size 1.016 1.016)) (justify right)))
@@
 (global_label "LED_CLOCK_B1_TO_C1" (shape passive) (at 180.34 38.1 0) (effects (font (size 1.016 1.016)) (justify right)))
 (global_label "LED_DATA_B1_TO_C1" (shape passive) (at 180.34 40.64 0) (effects (font (size 1.016 1.016)) (justify right)))
-(symbol (lib_id "Board:SK9822") (at 330.2 25.4 0) (unit 1) (in_bom yes) (on_board yes) (dnp no) (property "Reference" "U9" (at 330.2 20.32 0) (effects (font (size 1.27 1.27)))) (property "Value" "SK9822-A" (at 330.2 22.86 0) (effects (font (size 1.27 1.27)))) (property "Footprint" "" (at 330.2 25.4 0) (effects (font (size 1.27 1.27)) (hide yes))) (property "Datasheet" "https://www.rose-lighting.com/wp-content/uploads/sites/53/2020/05/SK9822-A-REV.01-EN-5050-RGB-27K-HZ-PWM-30M-bps-speed.pdf" (at 330.2 27.94 0) (effects (font (size 1.27 1.27)) (hide yes))) (property "Description" "Clocked 5050 RGB LED" (at 330.2 30.48 0) (effects (font (size 1.27 1.27)) (hide yes))) (instances (project "chess-board" (path "/78e160a7-634d-5fb3-901f-997b418a9dc6/b595d5f5-7ddb-5b0e-9c84-e831702cdbbb" (reference "U9") (unit 1)))))
+(symbol (lib_id "Board:SK9822") (at 330.2 25.4 0) (unit 1) (in_bom yes) (on_board yes) (dnp no) (property "Reference" "U9" (at 330.2 20.32 0) (effects (font (size 1.27 1.27)))) (property "Value" "SK9822-A" (at 330.2 22.86 0) (effects (font (size 1.27 1.27)))) (property "Footprint" "SK9822" (at 330.2 25.4 0) (effects (font (size 1.27 1.27)) (hide yes))) (property "Datasheet" "https://www.rose-lighting.com/wp-content/uploads/sites/53/2020/05/SK9822-A-REV.01-EN-5050-RGB-27K-HZ-PWM-30M-bps-speed.pdf" (at 330.2 27.94 0) (effects (font (size 1.27 1.27)) (hide yes))) (property "Description" "Clocked 5050 RGB LED" (at 330.2 30.48 0) (effects (font (size 1.27 1.27)) (hide yes))) (instances (project "chess-board" (path "/78e160a7-634d-5fb3-901f-997b418a9dc6/b595d5f5-7ddb-5b0e-9c84-e831702cdbbb" (reference "U9") (unit 1)))))
 (global_label "LED_DATA_D1_TO_E1" (shape passive) (at 307.34 27.94 0) (effects (font (size 1.016 1.016)) (justify right)))
 (global_label "LED_CLOCK_D1_TO_E1" (shape passive) (at 307.34 30.48 0) (effects (font (size 1.016 1.016)) (justify right)))
